Commit message: Simplify collision model

File: urdf/body/body.urdf.xacro (robot description, xacro)
@@ -13,10 +13,11 @@
       <visual>
         <geometry>
-          <mesh filename="package://raspimouse_description/meshes/dae/body/RasPiMouse_body.dae"/>
+          <mesh filename="package://raspimouse_description/meshes/dae/body/RasPiMouse_body.dae" />
         </geometry>
       </visual>
       <collision>
+        <origin rpy="0 0 0" xyz="0.005 0 0.040" />
         <geometry>
-          <mesh filename="package://raspimouse_description/meshes/dae/body/RasPiMouse_body.dae"/>
+          <box size="0.117 0.080 0.080"/>
         </geometry>
       </collision>

File: urdf/body/body_urg.urdf.xacro (robot description, xacro)
@@ -17,6 +17,9 @@
       </visual>
       <collision>
+        <!-- <origin rpy="0 0 ${radians(-90)}" /> -->
+        <origin rpy="0 0 0" xyz="0.005 0 0.0435" />
         <geometry>
-          <mesh filename="package://raspimouse_description/meshes/dae/body/RasPiMouse_body-TopPlate.dae"/>
+          <!-- <mesh filename="package://raspimouse_description/meshes/stl/collision/collision_body.stl" scale="0.001 0.001 0.00116" /> -->
+          <box size="0.117 0.080 0.087"/>
         </geometry>
       </collision>

File: urdf/sensors/lrf.urdf.xacro (robot description, xacro)
@@ -15,6 +15,7 @@
       </visual>
       <collision>
+        <origin xyz="0 0 -0.01815" />
         <geometry>
-          <mesh filename="package://raspimouse_description/meshes/dae/sensor/URG_center.dae"/>
+          <cylinder radius="0.025" length="0.070"/>
         </geometry>
       </collision>

File: urdf/wheel/wheel.urdf.xacro (robot description, xacro)
@@ -3,8 +3,7 @@
   <xacro:include filename="$(find raspimouse_description)/urdf/wheel/wheel.transmission.xacro"/>
   <xacro:include filename="$(find raspimouse_description)/urdf/wheel/wheel.gazebo.xacro"/>
-  <!-- <property name="wheel_radius" value="0.0239"/> -->
-  <property name="wheel_radius" value="0.0249"/>
-  <property name="wheel_length" value="0.01"/>
-  <property name="wheel_mass" value="0.0113"/>
+  <xacro:property name="wheel_radius" value="0.024"/>
+  <xacro:property name="wheel_length" value="0.010"/>
+  <xacro:property name="wheel_mass" value="0.0113"/>
   <xacro:macro name="wheel" params="prefix parent *joint_origin *joint_axis">
   <joint name="${prefix}_wheel_joint" type="continuous">
@@ -24,8 +23,7 @@
     </visual>
     <collision>
-      <!-- <insert_block name="joint_origin"/> -->
+      <origin xyz="0 0 0.003" />
         <geometry>
-          <!-- <cylinder radius="${wheel_radius}" length="${wheel_length}"/> -->
-          <mesh filename="package://raspimouse_description/meshes/dae/wheel/RasPiMouse_wheel.dae"/>
+          <cylinder radius="${wheel_radius}" length="${wheel_length}"/>
         </geometry>
     </collision>

Commit message: Add original collision geometry as comment

File: urdf/body/body.urdf.xacro (robot description, xacro)
@@ -17,4 +17,7 @@
       </visual>
       <collision>
+        <!-- <geometry> -->
+          <!-- <mesh filename="package://raspimouse_description/meshes/dae/body/RasPiMouse_body.dae" /> -->
+        <!-- </geometry> -->
         <origin rpy="0 0 0" xyz="0.005 0 0.040" />
         <geometry>

File: urdf/body/body_urg.urdf.xacro (robot description, xacro)
@@ -17,4 +17,7 @@
       </visual>
       <collision>
+        <!-- <geometry> -->
+          <!-- <mesh filename="package://raspimouse_description/meshes/dae/body/RasPiMouse_body-TopPlate.dae"/> -->
+        <!-- </geometry> -->
         <origin rpy="0 0 0" xyz="0.005 0 0.0435" />
         <geometry>

File: urdf/sensors/lrf.urdf.xacro (robot description, xacro)
@@ -15,4 +15,7 @@
       </visual>
       <collision>
+        <!-- <geometry> -->
+          <!-- <mesh filename="package://raspimouse_description/meshes/dae/sensor/URG_center.dae"/> -->
+        <!-- </geometry> -->
         <origin xyz="0 0 -0.01815" />
         <geometry>

File: urdf/wheel/wheel.urdf.xacro (robot description, xacro)
@@ -23,4 +23,7 @@
     </visual>
     <collision>
+      <!-- <geometry> -->
+        <!-- <mesh filename="package://raspimouse_description/meshes/dae/wheel/RasPiMouse_wheel.dae"/> -->
+      <!-- </geometry> -->
       <origin xyz="0 0 0.003" />
         <geometry>

Commit message: Simplify collision model (#16)
* Simplify collision model

* Remove unused comment

* Add original collision geometry as comment

File: urdf/body/body.urdf.xacro (robot description, xacro)
@@ -13,10 +13,14 @@
       <visual>
         <geometry>
-          <mesh filename="package://raspimouse_description/meshes/dae/body/RasPiMouse_body.dae"/>
+          <mesh filename="package://raspimouse_description/meshes/dae/body/RasPiMouse_body.dae" />
         </geometry>
       </visual>
       <collision>
+        <!-- <geometry> -->
+          <!-- <mesh filename="package://raspimouse_description/meshes/dae/body/RasPiMouse_body.dae" /> -->
+        <!-- </geometry> -->
+        <origin rpy="0 0 0" xyz="0.005 0 0.040" />
         <geometry>
-          <mesh filename="package://raspimouse_description/meshes/dae/body/RasPiMouse_body.dae"/>
+          <box size="0.117 0.080 0.080"/>
         </geometry>
       </collision>

File: urdf/body/body_urg.urdf.xacro (robot description, xacro)
@@ -17,6 +17,10 @@
       </visual>
       <collision>
+        <!-- <geometry> -->
+          <!-- <mesh filename="package://raspimouse_description/meshes/dae/body/RasPiMouse_body-TopPlate.dae"/> -->
+        <!-- </geometry> -->
+        <origin rpy="0 0 0" xyz="0.005 0 0.0435" />
         <geometry>
-          <mesh filename="package://raspimouse_description/meshes/dae/body/RasPiMouse_body-TopPlate.dae"/>
+          <box size="0.117 0.080 0.087"/>
         </geometry>
       </collision>

File: urdf/sensors/lrf.urdf.xacro (robot description, xacro)
@@ -15,6 +15,10 @@
       </visual>
       <collision>
+        <!-- <geometry> -->
+          <!-- <mesh filename="package://raspimouse_description/meshes/dae/sensor/URG_center.dae"/> -->
+        <!-- </geometry> -->
+        <origin xyz="0 0 -0.01815" />
         <geometry>
-          <mesh filename="package://raspimouse_description/meshes/dae/sensor/URG_center.dae"/>
+          <cylinder radius="0.025" length="0.070"/>
         </geometry>
       </collision>

File: urdf/wheel/wheel.urdf.xacro (robot description, xacro)
@@ -3,7 +3,6 @@
   <xacro:include filename="$(find raspimouse_description)/urdf/wheel/wheel.transmission.xacro"/>
   <xacro:include filename="$(find raspimouse_description)/urdf/wheel/wheel.gazebo.xacro"/>
-  <!-- <xacro:property name="wheel_radius" value="0.0239"/> -->
-  <xacro:property name="wheel_radius" value="0.0249"/>
-  <xacro:property name="wheel_length" value="0.01"/>
+  <xacro:property name="wheel_radius" value="0.024"/>
+  <xacro:property name="wheel_length" value="0.010"/>
   <xacro:property name="wheel_mass" value="0.0113"/>
   <xacro:macro name="wheel" params="prefix parent *joint_origin *joint_axis">
@@ -24,8 +23,10 @@
     </visual>
     <collision>
-      <!-- <xacro:insert_block name="joint_origin"/> -->
+      <!-- <geometry> -->
+        <!-- <mesh filename="package://raspimouse_description/meshes/dae/wheel/RasPiMouse_wheel.dae"/> -->
+      <!-- </geometry> -->
+      <origin xyz="0 0 0.003" />
         <geometry>
-          <!-- <cylinder radius="${wheel_radius}" length="${wheel_length}"/> -->
-          <mesh filename="package://raspimouse_description/meshes/dae/wheel/RasPiMouse_wheel.dae"/>
+          <cylinder radius="${wheel_radius}" length="${wheel_length}"/>
         </geometry>
     </collision>

Commit message: Update xacro for Gazebo simulator

File: urdf/body/body.urdf.xacro (robot description, xacro)
@@ -1,40 +1,55 @@
 <?xml version="1.0"?>
 <robot xmlns:xacro="http://ros.org/wiki/xacro">
-  <xacro:include filename="$(find raspimouse_description)/urdf/body/body.gazebo.xacro"/>
-  <xacro:property name="M_PI" value="3.1415926535897931" />
-  <xacro:property name="velocity_scale_factor" value="1.0"/>
-  <xacro:macro name="base" params="parent *joint_origin">
+  <xacro:macro name="base" params="parent lidar *joint_origin">
     <joint name="base_joint" type="fixed">
-      <xacro:insert_block name="joint_origin"/>
-      <parent link="${parent}"/>
-      <child link="base_link"/>
+      <xacro:insert_block name="joint_origin" />
+      <parent link="${parent}" />
+      <child link="base_link" />
     </joint>
     <link name="base_link">
-      <visual>
-        <geometry>
-          <mesh filename="package://raspimouse_description/meshes/dae/body/RasPiMouse_body.dae" />
-        </geometry>
-      </visual>
-      <collision>
-        <!-- <geometry> -->
-          <!-- <mesh filename="package://raspimouse_description/meshes/dae/body/RasPiMouse_body.dae" /> -->
-        <!-- </geometry> -->
-        <origin rpy="0 0 0" xyz="0.005 0 0.040" />
-        <geometry>
-          <box size="0.117 0.080 0.080"/>
-        </geometry>
-      </collision>
-      <inertial>
-        <!-- NOTE BEGINNING -->
-        <!-- Biased origin causes the slipping problem. -->
-        <!-- Not solved yet. -->
-        <!-- NOTE END -->
-        <!-- real origin -->
-        <!-- <origin xyz="&#45;0.005075 &#45;0.000427 0.029879"/> -->
-        <!-- virtual origin -->
-        <origin xyz="-0.001 0.0 0.029879"/>
-        <mass value="0.7186"/>
-        <inertia ixx="0.001238161833" ixy="0.000000904986" iyy="0.001368529369" ixz="0.000100297310" iyz="0.000022118177" izz="0.000784319117"/>
-      </inertial>
+      <xacro:if value="${lidar == 'none'}">
+        <visual>
+          <geometry>
+            <mesh filename="package://raspimouse_description/meshes/dae/body/RasPiMouse_body.dae" />
+          </geometry>
+        </visual>
+        <collision>
+          <!-- <geometry> -->
+            <!-- <mesh filename="package://raspimouse_description/meshes/dae/body/RasPiMouse_body.dae" /> -->
+          <!-- </geometry> -->
+          <origin rpy="0 0 0" xyz="0.005 0 0.040" />
+          <geometry>
+            <box size="0.117 0.080 0.080" />
+          </geometry>
+        </collision>
+        <inertial>
+          <origin xyz="-0.005075 -0.000427 0.029879" />
+          <mass value="0.7186" />
+          <inertia ixx="0.001238161833" ixy="0.000000904986" iyy="0.001368529369"
+                   ixz="0.000100297310" iyz="0.000022118177" izz="0.000784319117" />
+        </inertial>
+      </xacro:if>
+      <xacro:if value="${lidar == 'urg'}">
+        <visual>
+          <geometry>
+            <mesh filename="package://raspimouse_description/meshes/dae/body/RasPiMouse_body-TopPlate.dae"/>
+          </geometry>
+        </visual>
+        <collision>
+          <!-- <geometry> -->
+            <!-- <mesh filename="package://raspimouse_description/meshes/dae/body/RasPiMouse_body-TopPlate.dae" /> -->
+          <!-- </geometry> -->
+          <origin rpy="0 0 0" xyz="0.005 0 0.0435" />
+          <geometry>
+            <box size="0.117 0.080 0.087" />
+          </geometry>
+        </collision>
+        <inertial>
+          <origin xyz="-0.003851 -0.000443 0.031714" />
+          <mass value="0.759881"/>
+          <inertia ixx="0.001561279589" ixy="0.00000150035" iyy="0.001698462955"
+                   ixz="0.000042679786" iyz="0.000023629024" izz="0.000855782529"/>
+        </inertial>
+      </xacro:if>
     </link>
   </xacro:macro>

File: urdf/raspimouse.urdf.xacro (robot description, xacro)
@@ -5,62 +5,80 @@
        xmlns:interface="http://playerstage.sourceforge.net/gazebo/xmlschema/#interface"
        xmlns:xacro="http://ros.org/wiki/xacro">
-  <xacro:include filename="$(find raspimouse_description)/urdf/body/body.urdf.xacro"/>
-  <xacro:include filename="$(find raspimouse_description)/urdf/wheel/wheel.urdf.xacro"/>
-  <xacro:include filename="$(find raspimouse_description)/urdf/sensors/lightsens.urdf.xacro"/>
+  <xacro:arg name="lidar" default="none" />
+  <xacro:include filename="$(find raspimouse_description)/urdf/common.xacro" />
+  <xacro:include filename="$(find raspimouse_description)/urdf/body/body.urdf.xacro" />
+  <xacro:include filename="$(find raspimouse_description)/urdf/wheel/wheel.urdf.xacro" />
+  <xacro:include filename="$(find raspimouse_description)/urdf/sensors/lightsens.urdf.xacro" />
+  <xacro:include filename="$(find raspimouse_description)/urdf/sensors/lrf.urdf.xacro" />
   <!-- =============== Link & Joint =============== -->
   <!-- Base -->
-  <link name="base_footprint"/>
-  <xacro:base parent="base_footprint">
-    <origin xyz="0 0 0.00185"/>
+  <link name="base_footprint" />
+  <xacro:base parent="base_footprint" lidar="$(arg lidar)">
+    <origin xyz="0 0 0.00185" />
   </xacro:base>
   <!-- Wheel -->
   <xacro:wheel prefix="right" parent="base_link">
-    <origin xyz="0 -0.0425 0.02215" rpy="1.57 0 0"/>
-    <axis xyz="0 0 -1"/>
+    <origin xyz="0 -0.0425 0.02215" rpy="1.57 0 0" />
+    <axis xyz="0 0 -1" />
   </xacro:wheel>
   <xacro:wheel prefix="left" parent="base_link">
-    <origin xyz="0 0.0425 0.02215" rpy="-1.57 0 0"/>
-    <axis xyz="0 0 1"/>
+    <origin xyz="0 0.0425 0.02215" rpy="-1.57 0 0" />
+    <axis xyz="0 0 1" />
   </xacro:wheel>
   <!-- Sensors -->
   <xacro:light_sensor prefix="rf" parent="base_link">
-    <origin xyz="0.04 -0.045 0.032" rpy="0 0 0"/>
+    <origin xyz="0.04 -0.045 0.032" rpy="0 0 0" />
   </xacro:light_sensor>
   <xacro:light_sensor prefix="rs" parent="base_link">
-    <origin xyz="0.059 -0.01 0.032" rpy="0 0 -1.04"/>
+    <origin xyz="0.059 -0.01 0.032" rpy="0 0 -1.04" />
   </xacro:light_sensor>
   <xacro:light_sensor prefix="ls" parent="base_link">
-    <origin xyz="0.059 0.01 0.032" rpy="0 0 1.04"/>
+    <origin xyz="0.059 0.01 0.032" rpy="0 0 1.04" />
   </xacro:light_sensor>
   <xacro:light_sensor prefix="lf" parent="base_link">
-    <origin xyz="0.04 0.045 0.032" rpy="0 0 0"/>
+    <origin xyz="0.04 0.045 0.032" rpy="0 0 0" />
   </xacro:light_sensor>
-  <!-- ===============  Transmission =============== -->
-  <!-- PositionJointInterface: requires position -->
-  <!-- <xacro:wheel_trans prefix="right" interface="PositionJointInterface"/> -->
-  <!-- <xacro:wheel_trans prefix="left" interface="PositionJointInterface"/>  -->
-  <!-- VelocityJointInterface: requires position, velocity -->
-  <!-- for DiffDriveController -->
-  <xacro:wheel_trans prefix="right" interface="hardware_interface/VelocityJointInterface"/>
-  <xacro:wheel_trans prefix="left" interface="hardware_interface/VelocityJointInterface"/>
-  <!-- EffortJointInterface: requires position, velocity, effort -->
-  <!-- <xacro:wheel_trans prefix="right" interface="EffortJointInterface"/> -->
-  <!-- <xacro:wheel_trans prefix="left" interface="EffortJointInterface"/>  -->
+  <xacro:if value="${'$(arg lidar)' == 'urg'}">
+    <xacro:lrf_sensor prefix="urg_lrf_link" parent="base_link">
+      <origin xyz="0.0 0.0 0.14060" rpy="0 0 0" />
+    </xacro:lrf_sensor>
+  </xacro:if>
   <!-- =============== Gazebo =============== -->
   <gazebo>
-    <plugin name="gazebo_ros_control" filename="libgazebo_ros_control.so">
+    <plugin name="gazebo_ros_control" filename="libgazebo_ros_control.so" />
+  </gazebo>
+  <!-- Sensors -->
+  <xacro:lightsensor_gazebo prefix="rf" base_rad="0" rad_range="0.3" min_range="0.01" max_range="0.6" robot_namespace="raspimouse_on_gazebo" />
+  <xacro:lightsensor_gazebo prefix="rs" base_rad="-1.04" rad_range="0.3" min_range="0.01" max_range="0.6" robot_namespace="raspimouse_on_gazebo" />
+  <xacro:lightsensor_gazebo prefix="ls" base_rad="1.04" rad_range="0.3" min_range="0.01" max_range="0.6" robot_namespace="raspimouse_on_gazebo" />
+  <xacro:lightsensor_gazebo prefix="lf" base_rad="0" rad_range="0.3" min_range="0.01" max_range="0.6" robot_namespace="raspimouse_on_gazebo" />
+  <xacro:if value="${'$(arg lidar)' == 'urg'}">
+    <xacro:lrf_gazebo prefix="urg" base_rad="0" rad_range="4.71" min_range="0.10" max_range="5.6" />
+  </xacro:if>
+  <!-- DiffDriveController -->
+  <gazebo>
+    <plugin name="differential_drive_controller" filename="libgazebo_ros_diff_drive.so">
+      <alwaysOn>true</alwaysOn>
       <robotNamespace>raspimouse_on_gazebo</robotNamespace>
+      <updateRate>50</updateRate>
+      <legacyMode>false</legacyMode>
+      <leftJoint>left_wheel_joint</leftJoint>
+      <rightJoint>right_wheel_joint</rightJoint>
+      <robotBaseFrame>base_footprint</robotBaseFrame>
+      <wheelSeparation>${wheel_separation}</wheelSeparation>
+      <wheelDiameter>${wheel_radius*2.0}</wheelDiameter>
+      <publishWheelJointState>true</publishWheelJointState>
+      <rosDebugLevel>na</rosDebugLevel>
+      <commandTopic>cmd_vel</commandTopic>
+      <odometryTopic>odom</odometryTopic>
+      <odometryFrame>odom</odometryFrame>
+      <publishWheelTF>false</publishWheelTF>
+      <publishOdomTF>false</publishOdomTF>
+      <wheelAcceleration>0</wheelAcceleration>
+      <wheelTorque>5</wheelTorque>
+      <odometrySource>world</odometrySource>
+      <publishTf>1</publishTf>
     </plugin>
   </gazebo>
-  <!-- Base -->
-  <xacro:base_gazebo/>
-  <!-- Wheel -->
-  <xacro:wheel_gazebo prefix="right"/>
-  <xacro:wheel_gazebo prefix="left"/>
-  <!-- Sensors -->
-  <xacro:lightsensor_gazebo prefix="rf" base_rad="0" rad_range="0.3" min_range="0.01" max_range="0.6"/>
-  <xacro:lightsensor_gazebo prefix="rs" base_rad="-1.04" rad_range="0.3" min_range="0.01" max_range="0.6"/>
-  <xacro:lightsensor_gazebo prefix="ls" base_rad="1.04" rad_range="0.3" min_range="0.01" max_range="0.6"/>
-  <xacro:lightsensor_gazebo prefix="lf" base_rad="0" rad_range="0.3" min_range="0.01" max_range="0.6"/>
   <raspimouse_on_gazebo/>
 </robot>

File: urdf/sensors/lightsens.gazebo.xacro (robot description, xacro)
@@ -1,5 +1,5 @@
 <?xml version="1.0"?>
 <robot xmlns:xacro="http://ros.org/wiki/xacro">
-  <xacro:macro name="lightsensor_gazebo" params="prefix base_rad rad_range min_range max_range">
+  <xacro:macro name="lightsensor_gazebo" params="prefix base_rad rad_range min_range max_range robot_namespace">
     <gazebo reference="${prefix}">
       <sensor type="ray" name="${prefix}_lightsensor">
@@ -10,5 +10,4 @@
           <scan>
             <horizontal>
-              <!-- <samples>720</samples> -->
               <samples>1</samples>
               <resolution>1</resolution>
@@ -29,5 +28,6 @@
         </ray>
         <plugin name="gazebo_ros_${prefix}_lightsensor_controller" filename="libgazebo_ros_laser.so">
-          <topicName>/raspimouse_on_gazebo/${prefix}_scan</topicName>
+          <robotNamespace>${robot_namespace}</robotNamespace>
+          <topicName>${prefix}_scan</topicName>
           <frameName>${prefix}</frameName>
         </plugin>

File: urdf/sensors/lightsens.urdf.xacro (robot description, xacro)
@@ -1,10 +1,11 @@
 <?xml version="1.0"?>
 <robot name="light_sensor" xmlns:xacro="http://ros.org/wiki/xacro">
-  <xacro:include filename="$(find raspimouse_description)/urdf/sensors/lightsens.gazebo.xacro"/>
+  <xacro:include filename="$(find raspimouse_description)/urdf/common.xacro" />
+  <xacro:include filename="$(find raspimouse_description)/urdf/sensors/lightsens.gazebo.xacro" />
   <xacro:macro name="light_sensor" params="prefix parent *joint_origin">
     <joint name="${prefix}_joint" type="fixed">
-      <xacro:insert_block name="joint_origin"/>
-      <parent link="${parent}"/>
-      <child link="${prefix}"/>
+      <xacro:insert_block name="joint_origin" />
+      <parent link="${parent}" />
+      <child link="${prefix}" />
     </joint>
     <link name="${prefix}">
@@ -14,7 +15,5 @@
         </geometry>
       </visual>
-      <material name="grey">
-        <color rgba="0.5 0.5 0.5 1"/>
-      </material>
+      <material name="Gray" />
       <inertial>
         <mass value="0.000001" />
@@ -26,5 +25,5 @@
     </link>
     <!-- Set up laser gazebo details -->
-    <hokuyo_laser />
+    <!-- <hokuyo_laser /> -->
   </xacro:macro>
 </robot>

File: urdf/sensors/lrf.gazebo.xacro (robot description, xacro)
@@ -8,10 +8,8 @@
         <visualize>false</visualize>
         <update_rate>10</update_rate>
-        <!-- <update_rate>1</update_rate> -->
         <ray>
           <scan>
             <horizontal>
               <samples>720</samples>
-              <!-- <samples>10</samples> -->
               <resolution>1</resolution>
               <min_angle>${base_rad-rad_range/2}</min_angle>
@@ -31,6 +29,5 @@
         </ray>
         <plugin name="gazebo_ros_${prefix}_lrf_controller" filename="libgazebo_ros_laser.so">
-          <!-- <topicName>/hokuyo/${prefix}/scan</topicName> -->
-          <topicName>/scan</topicName>
+          <topicName>scan</topicName>
           <frameName>${prefix}_lrf_link</frameName>
         </plugin>

File: urdf/sensors/lrf.urdf.xacro (robot description, xacro)
@@ -1,4 +1,4 @@
 <?xml version="1.0"?>
-<robot name="light_sensor" xmlns:xacro="http://ros.org/wiki/xacro">
+<robot name="urg_sensor" xmlns:xacro="http://ros.org/wiki/xacro">
   <xacro:include filename="$(find raspimouse_description)/urdf/sensors/lrf.gazebo.xacro"/>
   <xacro:macro name="lrf_sensor" params="prefix parent *joint_origin">
@@ -27,10 +27,7 @@
         <origin xyz="0 0 0" />
         <inertia ixx="0.0001" ixy="0.0" ixz="0.0"
-          iyy="0.0001" iyz="0.0"
-          izz="0.0001" />
+          iyy="0.0001" iyz="0.0" izz="0.0001" />
       </inertial>
     </link>
-    <!-- Set up laser gazebo details -->
-    <hokuyo_laser />
   </xacro:macro>
 </robot>

File: urdf/wheel/wheel.urdf.xacro (robot description, xacro)
@@ -1,9 +1,5 @@
 <?xml version="1.0"?>
 <robot xmlns:xacro="http://ros.org/wiki/xacro">
-  <xacro:include filename="$(find raspimouse_description)/urdf/wheel/wheel.transmission.xacro"/>
-  <xacro:include filename="$(find raspimouse_description)/urdf/wheel/wheel.gazebo.xacro"/>
-  <xacro:property name="wheel_radius" value="0.024"/>
-  <xacro:property name="wheel_length" value="0.010"/>
-  <xacro:property name="wheel_mass" value="0.0113"/>
+  <xacro:include filename="$(find raspimouse_description)/urdf/common.xacro" />
   <xacro:macro name="wheel" params="prefix parent *joint_origin *joint_axis">
   <joint name="${prefix}_wheel_joint" type="continuous">
