Commit message: Update model and add RT Corporation logo

File: urdf/body/body.urdf.xacro (robot description, xacro)
@@ -8,35 +8,40 @@
     </joint>
     <link name="base_link">
-      <xacro:if value="${lidar == 'none'}">
+      <visual>
+        <geometry>
+          <mesh filename="package://raspimouse_description/meshes/dae/body/raspimouse_body.dae" />
+        </geometry>
+      </visual>
+      <collision>
+        <!-- <geometry> -->
+          <!-- <mesh filename="package://raspimouse_description/meshes/dae/body/raspimouse_body.dae" /> -->
+        <!-- </geometry> -->
+        <origin rpy="0 0 0" xyz="0.005 0 0.040" />
+        <geometry>
+          <box size="0.117 0.080 0.080" />
+        </geometry>
+      </collision>
+      <inertial>
+        <origin xyz="-0.005075 -0.000427 0.029879" />
+        <mass value="0.7186" />
+        <inertia ixx="0.001238161833" ixy="0.000000904986" iyy="0.001368529369"
+                  ixz="0.000100297310" iyz="0.000022118177" izz="0.000784319117" />
+      </inertial>
+    </link>
+    <xacro:if value="${lidar == 'urg'}">
+      <joint name="urg_mount_joint" type="fixed">
+        <origin rpy="0 0 0" xyz="0 0 0" />
+        <parent link="base_link" />
+        <child link="urg_mount_link" />
+      </joint>
+      <link name="urg_mount_link">
         <visual>
           <geometry>
-            <mesh filename="package://raspimouse_description/meshes/dae/body/RasPiMouse_body.dae" />
+            <mesh filename="package://raspimouse_description/meshes/dae/body/raspimouse_top_plate.dae"/>
           </geometry>
         </visual>
         <collision>
           <!-- <geometry> -->
-            <!-- <mesh filename="package://raspimouse_description/meshes/dae/body/RasPiMouse_body.dae" /> -->
-          <!-- </geometry> -->
-          <origin rpy="0 0 0" xyz="0.005 0 0.040" />
-          <geometry>
-            <box size="0.117 0.080 0.080" />
-          </geometry>
-        </collision>
-        <inertial>
-          <origin xyz="-0.005075 -0.000427 0.029879" />
-          <mass value="0.7186" />
-          <inertia ixx="0.001238161833" ixy="0.000000904986" iyy="0.001368529369"
-                   ixz="0.000100297310" iyz="0.000022118177" izz="0.000784319117" />
-        </inertial>
-      </xacro:if>
-      <xacro:if value="${lidar == 'urg'}">
-        <visual>
-          <geometry>
-            <mesh filename="package://raspimouse_description/meshes/dae/body/RasPiMouse_body-TopPlate.dae"/>
-          </geometry>
-        </visual>
-        <collision>
-          <!-- <geometry> -->
-            <!-- <mesh filename="package://raspimouse_description/meshes/dae/body/RasPiMouse_body-TopPlate.dae" /> -->
+            <!-- <mesh filename="package://raspimouse_description/meshes/dae/body/raspimouse_top_plate.dae" /> -->
           <!-- </geometry> -->
           <origin rpy="0 0 0" xyz="0.005 0 0.0435" />
@@ -51,6 +56,6 @@
                    ixz="0.000042679786" iyz="0.000023629024" izz="0.000855782529"/>
         </inertial>
-      </xacro:if>
-    </link>
+      </link>
+    </xacro:if>
   </xacro:macro>
 </robot>

File: urdf/raspimouse.urdf (robot description, URDF)
Before this commit: robot raspimouse, 4 links, 3 joints
Links:
- link base_link: geometry visual mesh filename=package://raspimouse_description/meshes/dae/body/raspiMouse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
- link left_wheel: geometry visual mesh filename=package://raspimouse_description/meshes/dae/wheel/raspiMous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
- link right_wheel: geometry visual mesh filename=package://raspimouse_description/meshes/dae/wheel/raspimous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

File: urdf/sensors/lrf.gazebo.xacro (robot description, xacro)
@@ -4,7 +4,6 @@
     <gazebo reference="${prefix}_lrf_link">
       <sensor type="ray" name="${prefix}_lrf_sensor">
-        <!-- <pose>0.0 0.0 0.05315 0 0 0</pose> -->
-        <pose>0 0 1 0 0 0</pose>
-        <visualize>false</visualize>
+        <pose>0 0 0 0 0 0</pose>
+        <visualize>$(arg laser_visual)</visualize>
         <update_rate>10</update_rate>
         <ray>

File: urdf/sensors/lrf.urdf.xacro (robot description, xacro)
@@ -2,4 +2,5 @@
 <robot name="urg_sensor" xmlns:xacro="http://ros.org/wiki/xacro">
   <xacro:include filename="$(find raspimouse_description)/urdf/sensors/lrf.gazebo.xacro"/>
+  <xacro:arg name="laser_visual" default="false"/>
   <xacro:macro name="lrf_sensor" params="prefix parent *joint_origin">
     <joint name="${prefix}_joint" type="fixed">
@@ -11,10 +12,10 @@
       <visual>
         <geometry>
-          <mesh filename="package://raspimouse_description/meshes/dae/sensor/URG_center.dae"/>
+          <mesh filename="package://raspimouse_description/meshes/dae/sensor/urg_optical_axis_center_origin.dae"/>
         </geometry>
       </visual>
       <collision>
         <!-- <geometry> -->
-          <!-- <mesh filename="package://raspimouse_description/meshes/dae/sensor/URG_center.dae"/> -->
+          <!-- <mesh filename="package://raspimouse_description/meshes/dae/sensor/urg_optical_axis_center_origin.dae"/> -->
         <!-- </geometry> -->
         <origin xyz="0 0 -0.01815" />

File: urdf/wheel/wheel.urdf.xacro (robot description, xacro)
@@ -15,10 +15,10 @@
     <visual>
       <geometry>
-        <mesh filename="package://raspimouse_description/meshes/dae/wheel/RasPiMouse_wheel.dae"/>
+        <mesh filename="package://raspimouse_description/meshes/dae/wheel/raspimouse_wheel.dae"/>
       </geometry>
     </visual>
     <collision>
       <!-- <geometry> -->
-        <!-- <mesh filename="package://raspimouse_description/meshes/dae/wheel/RasPiMouse_wheel.dae"/> -->
+        <!-- <mesh filename="package://raspimouse_description/meshes/dae/wheel/raspimouse_wheel.dae"/> -->
       <!-- </geometry> -->
       <origin xyz="0 0 0.003" />

Commit message: Separate option parts

File: urdf/body/body.urdf.xacro (robot description, xacro)
@@ -2,5 +2,5 @@
 <robot xmlns:xacro="http://ros.org/wiki/xacro">
   <xacro:include filename="$(find raspimouse_description)/urdf/body/body.gazebo.xacro" />
-  <xacro:macro name="base" params="parent lidar *joint_origin">
+  <xacro:macro name="base" params="parent *joint_origin">
     <joint name="base_joint" type="fixed">
       <xacro:insert_block name="joint_origin" />
@@ -32,33 +32,4 @@
       </inertial>
     </link>
-    <xacro:if value="${lidar == 'urg'}">
-      <joint name="urg_mount_joint" type="fixed">
-        <origin rpy="0 0 0" xyz="0 0 0" />
-        <parent link="base_link" />
-        <child link="urg_mount_link" />
-      </joint>
-      <link name="urg_mount_link">
-        <visual>
-          <geometry>
-            <mesh filename="package://raspimouse_description/meshes/dae/body/raspimouse_top_plate.dae" />
-          </geometry>
-        </visual>
-        <collision>
-          <!-- <geometry> -->
-            <!-- <mesh filename="package://raspimouse_description/meshes/dae/body/raspimouse_top_plate.dae" /> -->
-          <!-- </geometry> -->
-          <origin rpy="0 0 0" xyz="0.005 0 0.0435" />
-          <geometry>
-            <box size="0.117 0.080 0.087" />
-          </geometry>
-        </collision>
-        <inertial>
-          <origin xyz="-0.003851 -0.000443 0.031714" />
-          <mass value="0.759881" />
-          <inertia ixx="0.001561279589" ixy="0.00000150035" iyy="0.001698462955"
-                   ixz="0.000042679786" iyz="0.000023629024" izz="0.000855782529" />
-        </inertial>
-      </link>
-    </xacro:if>
   </xacro:macro>
 </robot>

File: urdf/raspimouse.urdf.xacro (robot description, xacro)
@@ -16,4 +16,5 @@
   <xacro:include filename="$(find raspimouse_description)/urdf/common.xacro" />
   <xacro:include filename="$(find raspimouse_description)/urdf/body/body.urdf.xacro" />
+  <xacro:include filename="$(find raspimouse_description)/urdf/body/option.urdf.xacro" />
   <xacro:include filename="$(find raspimouse_description)/urdf/wheel/wheel.urdf.xacro" />
   <xacro:include filename="$(find raspimouse_description)/urdf/wheel/diffdrive.gazebo.xacro" />
@@ -23,5 +24,5 @@
   <!-- Base -->
   <link name="base_footprint" />
-  <xacro:base parent="base_footprint" lidar="$(arg lidar)">
+  <xacro:base parent="base_footprint">
     <origin xyz="0 0 0.00185" />
   </xacro:base>
@@ -49,5 +50,8 @@
   </xacro:light_sensor>
   <xacro:if value="${'$(arg lidar)' == 'urg'}">
-    <xacro:lidar_urg_sensor sensor_link_name="$(arg lidar_frame)" parent="base_link">
+    <xacro:lidar_urg_mount prefix="urg_mount" parent="base_link">
+      <origin xyz="0 0 0" rpy="0 0 0" />
+    </xacro:lidar_urg_mount>
+    <xacro:lidar_urg_sensor sensor_link_name="$(arg lidar_frame)" parent="urg_mount_link">
       <origin xyz="0.0 0.0 0.14060" rpy="0 0 0" />
     </xacro:lidar_urg_sensor>

Commit message: Separate option parts

File: urdf/body/body.urdf.xacro (robot description, xacro)
@@ -2,5 +2,5 @@
 <robot xmlns:xacro="http://ros.org/wiki/xacro">
   <xacro:include filename="$(find raspimouse_description)/urdf/body/body.gazebo.xacro" />
-  <xacro:macro name="base" params="parent lidar *joint_origin">
+  <xacro:macro name="base" params="parent *joint_origin">
     <joint name="base_joint" type="fixed">
       <xacro:insert_block name="joint_origin" />
@@ -9,50 +9,26 @@
     </joint>
     <link name="base_link">
-      <xacro:if value="${lidar == 'none'}">
-        <visual>
-          <geometry>
-            <mesh filename="package://raspimouse_description/meshes/dae/body/RasPiMouse_body.dae" />
-          </geometry>
-        </visual>
-        <collision>
-          <!-- <geometry> -->
-            <!-- <mesh filename="package://raspimouse_description/meshes/dae/body/RasPiMouse_body.dae" /> -->
-          <!-- </geometry> -->
-          <origin rpy="0 0 0" xyz="0.005 0 0.040" />
-          <geometry>
-            <box size="0.117 0.080 0.080" />
-          </geometry>
-        </collision>
-        <inertial>
-          <origin xyz="-0.005075 0.0 0.03" />
-          <mass value="0.7186" />
-          <xacro:box_inertia m="0.7" x="0.1" y="0.08" z="0.08" />
-          <!-- <origin xyz="-0.005075 -0.000427 0.029879" /> -->
-          <!-- <inertia ixx="0.001238161833" ixy="0.000000904986" iyy="0.001368529369"
+      <visual>
+        <geometry>
+          <mesh filename="package://raspimouse_description/meshes/dae/body/RasPiMouse_body.dae" />
+        </geometry>
+      </visual>
+      <collision>
+        <!-- <geometry> -->
+        <!-- <mesh filename="package://raspimouse_description/meshes/dae/body/RasPiMouse_body.dae" /> -->
+        <!-- </geometry> -->
+        <origin rpy="0 0 0" xyz="0.005 0 0.040" />
+        <geometry>
+          <box size="0.117 0.080 0.080" />
+        </geometry>
+      </collision>
+      <inertial>
+        <origin xyz="-0.005075 0.0 0.03" />
+        <mass value="0.7186" />
+        <xacro:box_inertia m="0.7" x="0.1" y="0.08" z="0.08" />
+        <!-- <origin xyz="-0.005075 -0.000427 0.029879" /> -->
+        <!-- <inertia ixx="0.001238161833" ixy="0.000000904986" iyy="0.001368529369"
                     ixz="0.000100297310" iyz="0.000022118177" izz="0.000784319117" /> -->
-        </inertial>
-      </xacro:if>
-      <xacro:if value="${lidar == 'urg'}">
-        <visual>
-          <geometry>
-            <mesh filename="package://raspimouse_description/meshes/dae/body/RasPiMouse_body-TopPlate.dae"/>
-          </geometry>
-        </visual>
-        <collision>
-          <!-- <geometry> -->
-            <!-- <mesh filename="package://raspimouse_description/meshes/dae/body/RasPiMouse_body-TopPlate.dae" /> -->
-          <!-- </geometry> -->
-          <origin rpy="0 0 0" xyz="0.005 0 0.0435" />
-          <geometry>
-            <box size="0.117 0.080 0.087" />
-          </geometry>
-        </collision>
-        <inertial>
-          <origin xyz="-0.003851 -0.000443 0.031714" />
-          <mass value="0.759881" />
-          <inertia ixx="0.001561279589" ixy="0.00000150035" iyy="0.001698462955"
-                   ixz="0.000042679786" iyz="0.000023629024" izz="0.000855782529" />
-        </inertial>
-      </xacro:if>
+      </inertial>
     </link>
   </xacro:macro>

File: urdf/raspimouse.urdf.xacro (robot description, xacro)
@@ -15,4 +15,5 @@
   <xacro:include filename="$(find raspimouse_description)/urdf/common.xacro" />
   <xacro:include filename="$(find raspimouse_description)/urdf/body/body.urdf.xacro" />
+  <xacro:include filename="$(find raspimouse_description)/urdf/body/option.urdf.xacro" />
   <xacro:include filename="$(find raspimouse_description)/urdf/wheel/wheel.urdf.xacro" />
   <xacro:include filename="$(find raspimouse_description)/urdf/wheel/diffdrive.gazebo.xacro" />
@@ -22,5 +23,5 @@
   <!-- Base -->
   <link name="base_footprint" />
-  <xacro:base parent="base_footprint" lidar="$(arg lidar)">
+  <xacro:base parent="base_footprint">
     <origin xyz="0 0 0.00185" />
   </xacro:base>
@@ -48,5 +49,8 @@
   </xacro:light_sensor>
   <xacro:if value="${'$(arg lidar)' == 'urg'}">
-    <xacro:lidar_urg_sensor sensor_link_name="$(arg lidar_frame)" parent="base_link">
+    <xacro:lidar_urg_mount prefix="urg_mount" parent="base_link">
+      <origin xyz="0 0 0" rpy="0 0 0" />
+    </xacro:lidar_urg_mount>
+    <xacro:lidar_urg_sensor sensor_link_name="$(arg lidar_frame)" parent="urg_mount_link">
       <origin xyz="0.0 0.0 0.14060" rpy="0 0 0" />
     </xacro:lidar_urg_sensor>

Commit message: Avoid slipping

File: urdf/body/body.urdf.xacro (robot description, xacro)
@@ -1,4 +1,5 @@
 <?xml version="1.0"?>
 <robot xmlns:xacro="http://ros.org/wiki/xacro">
+  <xacro:include filename="$(find raspimouse_description)/urdf/body/body.gazebo.xacro" />
   <xacro:macro name="base" params="parent lidar *joint_origin">
     <joint name="base_joint" type="fixed">
@@ -23,8 +24,10 @@
       </collision>
       <inertial>
-        <origin xyz="-0.005075 -0.000427 0.029879" />
         <mass value="0.7186" />
-        <inertia ixx="0.001238161833" ixy="0.000000904986" iyy="0.001368529369"
-                  ixz="0.000100297310" iyz="0.000022118177" izz="0.000784319117" />
+        <origin xyz="-0.005075 0.0 0.03" />
+        <xacro:box_inertia m="0.7" x="0.1" y="0.08" z="0.08" />
+        <!-- <origin xyz="-0.005075 -0.000427 0.029879" /> -->
+        <!-- <inertia ixx="0.001238161833" ixy="0.000000904986" iyy="0.001368529369"
+                  ixz="0.000100297310" iyz="0.000022118177" izz="0.000784319117" /> -->
       </inertial>
     </link>
@@ -38,5 +41,5 @@
         <visual>
           <geometry>
-            <mesh filename="package://raspimouse_description/meshes/dae/body/raspimouse_top_plate.dae"/>
+            <mesh filename="package://raspimouse_description/meshes/dae/body/raspimouse_top_plate.dae" />
           </geometry>
         </visual>
@@ -52,7 +55,7 @@
         <inertial>
           <origin xyz="-0.003851 -0.000443 0.031714" />
-          <mass value="0.759881"/>
+          <mass value="0.759881" />
           <inertia ixx="0.001561279589" ixy="0.00000150035" iyy="0.001698462955"
-                   ixz="0.000042679786" iyz="0.000023629024" izz="0.000855782529"/>
+                   ixz="0.000042679786" iyz="0.000023629024" izz="0.000855782529" />
         </inertial>
       </link>

File: urdf/wheel/wheel.urdf.xacro (robot description, xacro)
@@ -3,34 +3,44 @@
   <xacro:include filename="$(find raspimouse_description)/urdf/common.xacro" />
   <xacro:macro name="wheel" params="prefix parent *joint_origin *joint_axis">
-  <joint name="${prefix}_wheel_joint" type="continuous">
-    <xacro:insert_block name="joint_origin"/>
-    <xacro:insert_block name="joint_axis"/>
-    <parent link="${parent}"/>
-    <child link="${prefix}_wheel"/>
-    <limit effort="70" velocity="15"/>
-    <safety_controller  k_velocity="10" />
-    <dynamics damping="1.0" friction="1.0" />
-  </joint>
-  <link name="${prefix}_wheel">
-    <visual>
-      <geometry>
-        <mesh filename="package://raspimouse_description/meshes/dae/wheel/raspimouse_wheel.dae"/>
-      </geometry>
-    </visual>
-    <collision>
-      <!-- <geometry> -->
+    <joint name="${prefix}_wheel_joint" type="continuous">
+      <xacro:insert_block name="joint_origin" />
+      <xacro:insert_block name="joint_axis" />
+      <parent link="${parent}" />
+      <child link="${prefix}_wheel" />
+      <limit effort="70" velocity="15" />
+      <safety_controller k_velocity="10" />
+      <dynamics damping="1.0" friction="1.0" />
+    </joint>
+    <link name="${prefix}_wheel">
+      <visual>
+        <geometry>
+          <mesh filename="package://raspimouse_description/meshes/dae/wheel/raspimouse_wheel.dae" />
+        </geometry>
+      </visual>
+      <collision>
+        <!-- <geometry> -->
         <!-- <mesh filename="package://raspimouse_description/meshes/dae/wheel/raspimouse_wheel.dae"/> -->
-      <!-- </geometry> -->
-      <origin xyz="0 0 0.003" />
+        <!-- </geometry> -->
+        <origin xyz="0 0 0.003" />
         <geometry>
-          <cylinder radius="${wheel_radius}" length="${wheel_length}"/>
+          <cylinder radius="${wheel_radius}" length="${wheel_length}" />
         </geometry>
-    </collision>
+        <surface>
+          <friction>
+            <ode>
+              <mu>2</mu>
+              <mu2>2</mu2>
+              <slip1>0</slip1>
+              <slip2>0</slip2>
+            </ode>
+          </friction>
+        </surface>
+      </collision>
       <inertial>
-        <origin xyz="-0.000107 0 0.002875"/>
-        <mass value="${wheel_mass}"/>
-        <inertia ixx="0.000002208187" ixy="0.000000000001" iyy="0.00000218412" ixz="0.000000004787" iyz="0.000000000003" izz="0.000004078299"/>
+        <origin xyz="-0.000107 0 0.002875" />
+        <mass value="${wheel_mass}" />
+        <inertia ixx="0.000002208187" ixy="0.000000000001" iyy="0.00000218412" ixz="0.000000004787" iyz="0.000000000003" izz="0.000004078299" />
       </inertial>
-  </link>
+    </link>
   </xacro:macro>
 </robot>

Commit message: Avoid slipping

File: urdf/body/body.urdf.xacro (robot description, xacro)
@@ -1,4 +1,5 @@
 <?xml version="1.0"?>
 <robot xmlns:xacro="http://ros.org/wiki/xacro">
+  <xacro:include filename="$(find raspimouse_description)/urdf/body/body.gazebo.xacro" />
   <xacro:macro name="base" params="parent lidar *joint_origin">
     <joint name="base_joint" type="fixed">
@@ -24,8 +25,10 @@
         </collision>
         <inertial>
-          <origin xyz="-0.005075 -0.000427 0.029879" />
+          <origin xyz="-0.005075 0.0 0.03" />
           <mass value="0.7186" />
-          <inertia ixx="0.001238161833" ixy="0.000000904986" iyy="0.001368529369"
-                   ixz="0.000100297310" iyz="0.000022118177" izz="0.000784319117" />
+          <xacro:box_inertia m="0.7" x="0.1" y="0.08" z="0.08" />
+          <!-- <origin xyz="-0.005075 -0.000427 0.029879" /> -->
+          <!-- <inertia ixx="0.001238161833" ixy="0.000000904986" iyy="0.001368529369"
+                    ixz="0.000100297310" iyz="0.000022118177" izz="0.000784319117" /> -->
         </inertial>
       </xacro:if>
@@ -47,7 +50,7 @@
         <inertial>
           <origin xyz="-0.003851 -0.000443 0.031714" />
-          <mass value="0.759881"/>
+          <mass value="0.759881" />
           <inertia ixx="0.001561279589" ixy="0.00000150035" iyy="0.001698462955"
-                   ixz="0.000042679786" iyz="0.000023629024" izz="0.000855782529"/>
+                   ixz="0.000042679786" iyz="0.000023629024" izz="0.000855782529" />
         </inertial>
       </xacro:if>

File: urdf/wheel/wheel.urdf.xacro (robot description, xacro)
@@ -24,13 +24,23 @@
       <origin xyz="0 0 0.003" />
         <geometry>
-          <cylinder radius="${wheel_radius}" length="${wheel_length}"/>
+          <cylinder radius="${wheel_radius}" length="${wheel_length}" />
         </geometry>
-    </collision>
+        <surface>
+          <friction>
+            <ode>
+              <mu>2</mu>
+              <mu2>2</mu2>
+              <slip1>0</slip1>
+              <slip2>0</slip2>
+            </ode>
+          </friction>
+        </surface>
+      </collision>
       <inertial>
-        <origin xyz="-0.000107 0 0.002875"/>
-        <mass value="${wheel_mass}"/>
-        <inertia ixx="0.000002208187" ixy="0.000000000001" iyy="0.00000218412" ixz="0.000000004787" iyz="0.000000000003" izz="0.000004078299"/>
+        <origin xyz="-0.000107 0 0.002875" />
+        <mass value="${wheel_mass}" />
+        <inertia ixx="0.000002208187" ixy="0.000000000001" iyy="0.00000218412" ixz="0.000000004787" iyz="0.000000000003" izz="0.000004078299" />
       </inertial>
-  </link>
+    </link>
   </xacro:macro>
 </robot>
