Commit message: Fix slipping (#28)
* Fix wheel link missing problem

Also, add comments about params

-wheelTorque: 5
+wheelTorque: 500

Co-authored-by: Shota Aoki <s.aoki@rt-net.jp>

* Fix typo to suppress warnings loading GazeboPlugin

same as https://github.com/rt-net/jnmouse_description/pull/9

* Fix default namespace to avoid odometry tf error

related: https://github.com/rt-net/raspimouse_sim/pull/55

* Refactor

* Add an option to load gazebo plugin to allow URDF to be loaded without gazebo_ros

* Separate DiffDriveController into separate files

* Add laser link option

* s/laser_frame/lidar_frame/g

* Update lidar_frame name option

* Avoid slipping

* Separate option parts

Co-authored-by: Shota Aoki <s.aoki@rt-net.jp>

File: urdf/body/body.urdf.xacro (robot description, xacro)
@@ -1,5 +1,6 @@
 <?xml version="1.0"?>
 <robot xmlns:xacro="http://ros.org/wiki/xacro">
-  <xacro:macro name="base" params="parent lidar *joint_origin">
+  <xacro:include filename="$(find raspimouse_description)/urdf/body/body.gazebo.xacro" />
+  <xacro:macro name="base" params="parent *joint_origin">
     <joint name="base_joint" type="fixed">
       <xacro:insert_block name="joint_origin" />
@@ -8,48 +9,26 @@
     </joint>
     <link name="base_link">
-      <xacro:if value="${lidar == 'none'}">
-        <visual>
-          <geometry>
-            <mesh filename="package://raspimouse_description/meshes/dae/body/RasPiMouse_body.dae" />
-          </geometry>
-        </visual>
-        <collision>
-          <!-- <geometry> -->
-            <!-- <mesh filename="package://raspimouse_description/meshes/dae/body/RasPiMouse_body.dae" /> -->
-          <!-- </geometry> -->
-          <origin rpy="0 0 0" xyz="0.005 0 0.040" />
-          <geometry>
-            <box size="0.117 0.080 0.080" />
-          </geometry>
-        </collision>
-        <inertial>
-          <origin xyz="-0.005075 -0.000427 0.029879" />
-          <mass value="0.7186" />
-          <inertia ixx="0.001238161833" ixy="0.000000904986" iyy="0.001368529369"
-                   ixz="0.000100297310" iyz="0.000022118177" izz="0.000784319117" />
-        </inertial>
-      </xacro:if>
-      <xacro:if value="${lidar == 'urg'}">
-        <visual>
-          <geometry>
-            <mesh filename="package://raspimouse_description/meshes/dae/body/RasPiMouse_body-TopPlate.dae"/>
-          </geometry>
-        </visual>
-        <collision>
-          <!-- <geometry> -->
-            <!-- <mesh filename="package://raspimouse_description/meshes/dae/body/RasPiMouse_body-TopPlate.dae" /> -->
-          <!-- </geometry> -->
-          <origin rpy="0 0 0" xyz="0.005 0 0.0435" />
-          <geometry>
-            <box size="0.117 0.080 0.087" />
-          </geometry>
-        </collision>
-        <inertial>
-          <origin xyz="-0.003851 -0.000443 0.031714" />
-          <mass value="0.759881"/>
-          <inertia ixx="0.001561279589" ixy="0.00000150035" iyy="0.001698462955"
-                   ixz="0.000042679786" iyz="0.000023629024" izz="0.000855782529"/>
-        </inertial>
-      </xacro:if>
+      <visual>
+        <geometry>
+          <mesh filename="package://raspimouse_description/meshes/dae/body/RasPiMouse_body.dae" />
+        </geometry>
+      </visual>
+      <collision>
+        <!-- <geometry> -->
+        <!-- <mesh filename="package://raspimouse_description/meshes/dae/body/RasPiMouse_body.dae" /> -->
+        <!-- </geometry> -->
+        <origin rpy="0 0 0" xyz="0.005 0 0.040" />
+        <geometry>
+          <box size="0.117 0.080 0.080" />
+        </geometry>
+      </collision>
+      <inertial>
+        <origin xyz="-0.005075 0.0 0.03" />
+        <mass value="0.7186" />
+        <xacro:box_inertia m="0.7" x="0.1" y="0.08" z="0.08" />
+        <!-- <origin xyz="-0.005075 -0.000427 0.029879" /> -->
+        <!-- <inertia ixx="0.001238161833" ixy="0.000000904986" iyy="0.001368529369"
+                    ixz="0.000100297310" iyz="0.000022118177" izz="0.000784319117" /> -->
+      </inertial>
     </link>
   </xacro:macro>

Commit message: Fix merge error
https://github.com/rt-net/raspimouse_description/pull/29/commits/a25febe1c1cb9f722f22df125bd846d93efb01f1

File: urdf/body/body.urdf.xacro (robot description, xacro)
@@ -24,8 +24,10 @@
       </collision>
       <inertial>
-        <origin xyz="-0.005075 -0.000427 0.029879" />
+        <origin xyz="-0.005075 0.0 0.03" />
         <mass value="0.7186" />
-        <inertia ixx="0.001238161833" ixy="0.000000904986" iyy="0.001368529369"
-                  ixz="0.000100297310" iyz="0.000022118177" izz="0.000784319117" />
+        <xacro:box_inertia m="0.7" x="0.1" y="0.08" z="0.08" />
+        <!-- <origin xyz="-0.005075 -0.000427 0.029879" /> -->
+        <!-- <inertia ixx="0.001238161833" ixy="0.000000904986" iyy="0.001368529369"
+                    ixz="0.000100297310" iyz="0.000022118177" izz="0.000784319117" /> -->
       </inertial>
     </link>

Commit message: Update model and add RT Corporation logo (#29)
* Update model and add RT Corporation logo

* Fix main circuit board position

* Update xacro option

* Fix merge error

https://github.com/rt-net/raspimouse_description/pull/29/commits/a25febe1c1cb9f722f22df125bd846d93efb01f1

* Refactor

* Optimize collada

* Add URDF with URG

File: urdf/body/body.urdf.xacro (robot description, xacro)
@@ -11,10 +11,10 @@
       <visual>
         <geometry>
-          <mesh filename="package://raspimouse_description/meshes/dae/body/RasPiMouse_body.dae" />
+          <mesh filename="package://raspimouse_description/meshes/dae/body/raspimouse_body.dae" />
         </geometry>
       </visual>
       <collision>
         <!-- <geometry> -->
-        <!-- <mesh filename="package://raspimouse_description/meshes/dae/body/RasPiMouse_body.dae" /> -->
+          <!-- <mesh filename="package://raspimouse_description/meshes/dae/body/raspimouse_body.dae" /> -->
         <!-- </geometry> -->
         <origin rpy="0 0 0" xyz="0.005 0 0.040" />

File: urdf/body/option.urdf.xacro (robot description, xacro)
@@ -10,10 +10,10 @@
       <visual>
         <geometry>
-          <mesh filename="package://raspimouse_description/meshes/dae/body/RasPiMouse_TopPlate.dae"/>
+          <mesh filename="package://raspimouse_description/meshes/dae/body/raspimouse_top_plate.dae"/>
         </geometry>
       </visual>
       <collision>
         <!-- <geometry> -->
-          <!-- <mesh filename="package://raspimouse_description/meshes/dae/body/RasPiMouse_TopPlate.dae"/> -->
+          <!-- <mesh filename="package://raspimouse_description/meshes/dae/body/raspimouse_top_plate.dae"/> -->
         <!-- </geometry> -->
         <origin rpy="0 0 0" xyz="0.005 0 0.0435" />

File: urdf/raspimouse_with_urg.urdf (robot description, URDF)
Before this commit: robot raspimouse, 4 links, 3 joints
Links:
- added link lidar_link; visual mesh filename=package://raspimouse_description/meshes/dae/sensor/urg_opti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
- added link urg_mount_link; visual mesh filename=package://raspimouse_description/meshes/dae/body/raspimouse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
Joints:
- added joint urg_joint: type fixed, parent urg_mount_link, child lidar_link, origin xyz=0.0 0.0 0.14060 rpy=0 0 0
- added joint urg_mount_joint: type fixed, parent base_link, child urg_mount_link, origin xyz=0 0 0 rpy=0 0 0

File: urdf/sensors/lidar.gazebo.xacro (robot description, xacro)
@@ -5,5 +5,5 @@
       <sensor type="ray" name="${sensor_link_name}_sensor">
         <pose>0 0 0 0 0 0</pose>
-        <visualize>false</visualize>
+        <visualize>$(arg laser_visual)</visualize>
         <update_rate>10</update_rate>
         <ray>

File: urdf/sensors/lidar.urdf.xacro (robot description, xacro)
@@ -2,4 +2,5 @@
 <robot name="urg_sensor" xmlns:xacro="http://ros.org/wiki/xacro">
   <xacro:include filename="$(find raspimouse_description)/urdf/sensors/lidar.gazebo.xacro"/>
+  <xacro:arg name="laser_visual" default="false"/>
   <xacro:macro name="lidar_urg_sensor" params="sensor_link_name parent *joint_origin">
     <joint name="${sensor_link_name}_joint" type="fixed">
@@ -11,10 +12,10 @@
       <visual>
         <geometry>
-          <mesh filename="package://raspimouse_description/meshes/dae/sensor/URG_center.dae"/>
+          <mesh filename="package://raspimouse_description/meshes/dae/sensor/urg_optical_axis_center_origin.dae"/>
         </geometry>
       </visual>
       <collision>
         <!-- <geometry> -->
-          <!-- <mesh filename="package://raspimouse_description/meshes/dae/sensor/URG_center.dae"/> -->
+          <!-- <mesh filename="package://raspimouse_description/meshes/dae/sensor/urg_optical_axis_center_origin.dae"/> -->
         <!-- </geometry> -->
         <origin xyz="0 0 -0.01815" />

File: urdf/wheel/wheel.urdf.xacro (robot description, xacro)
@@ -15,10 +15,10 @@
     <visual>
       <geometry>
-        <mesh filename="package://raspimouse_description/meshes/dae/wheel/RasPiMouse_wheel.dae"/>
+        <mesh filename="package://raspimouse_description/meshes/dae/wheel/raspimouse_wheel.dae"/>
       </geometry>
     </visual>
     <collision>
       <!-- <geometry> -->
-        <!-- <mesh filename="package://raspimouse_description/meshes/dae/wheel/RasPiMouse_wheel.dae"/> -->
+        <!-- <mesh filename="package://raspimouse_description/meshes/dae/wheel/raspimouse_wheel.dae"/> -->
       <!-- </geometry> -->
       <origin xyz="0 0 0.003" />
