Commit message: Add web camera option

File: urdf/body/option.urdf.xacro (robot description, xacro)
@@ -29,3 +29,30 @@
     </link>
   </xacro:macro>
+  <xacro:macro name="camera_mount" params="prefix parent *joint_origin">
+    <joint name="${prefix}_joint" type="fixed">
+      <xacro:insert_block name="joint_origin" />
+      <parent link="${parent}" />
+      <child link="${prefix}_link" />
+    </joint>
+    <link name="${prefix}_link">
+      <visual>
+        <geometry>
+          <mesh filename="package://raspimouse_description/meshes/dae/body/raspimouse_camera_mount.dae" />
+        </geometry>
+      </visual>
+      <collision>
+        <!-- <geometry> -->
+        <!-- <mesh filename="package://raspimouse_description/meshes/dae/body/raspimouse_camera_mount.dae" /> -->
+        <!-- </geometry> -->
+        <origin rpy="0 0 0" xyz="-0.006 0 0" />
+        <geometry>
+          <box size="0.03 0.068 0.0016" />
+        </geometry>
+      </collision>
+      <inertial>
+        <mass value="0.005" />
+        <xacro:box_inertia m="0.005" x="0.05" y="0.07" z="0.002" />
+      </inertial>
+    </link>
+  </xacro:macro>
 </robot>

File: urdf/raspimouse.urdf.xacro (robot description, xacro)
@@ -8,4 +8,6 @@
   <xacro:arg name="lidar_frame" default="laser" />
   <xacro:arg name="laser_visual" default="true"/>
+  <xacro:arg name="camera" default="false" />
+  <xacro:arg name="camera_visual" default="false"/>
   <xacro:arg name="gazebo_plugin" default="false" />
   <xacro:arg name="tf" default="true" />
@@ -13,4 +15,5 @@
   <xacro:arg name="robot_namespace" default="/" />
   <xacro:arg name="diffdrive_namespace" default="/" />
+  <xacro:arg name="camera_namespace" default="/" />
   <xacro:arg name="sensor_namespace" default="raspimouse_on_gazebo" />
   <xacro:include filename="$(find raspimouse_description)/urdf/common.xacro" />
@@ -21,4 +24,5 @@
   <xacro:include filename="$(find raspimouse_description)/urdf/sensors/lightsens.urdf.xacro" />
   <xacro:include filename="$(find raspimouse_description)/urdf/sensors/lidar.urdf.xacro" />
+  <xacro:include filename="$(find raspimouse_description)/urdf/camera/camera.urdf.xacro" />
   <!-- =============== Link & Joint =============== -->
   <!-- Base -->
@@ -57,4 +61,12 @@
     </xacro:lidar_urg_sensor>
   </xacro:if>
+  <xacro:if value="$(arg camera)">
+    <xacro:camera_mount prefix="camera_mount" parent="base_link">
+      <origin rpy="0 0 0" xyz="0.085 0 0.0493" />
+    </xacro:camera_mount>
+    <xacro:webcam prefix="webcam" parent="camera_mount_link">
+      <origin xyz="0 0 0.01" rpy="0 0 0" />
+    </xacro:webcam>
+  </xacro:if>
   <!-- =============== Gazebo =============== -->
   <xacro:if value="$(arg gazebo_plugin)">
@@ -84,4 +96,9 @@
       <xacro:lidar_gazebo sensor_link_name="$(arg lidar_frame)" base_rad="0" rad_range="4.71" min_range="0.10" max_range="5.6" />
     </xacro:if>
+    <xacro:if value="$(arg camera)">
+      <xacro:camera_gazebo camera_name="webcam" camera_link="webcam_link"
+        robot_namespace="$(arg camera_namespace)"
+        robotdescription_namespace="/" />
+    </xacro:if>
     <!-- DiffDriveController -->
     <xacro:diffdrive_gazebo publish_tf="$(arg tf)" publish_jointstate="$(arg jointstate)"

Commit message: Adds macro lidar_multi_mount

File: urdf/body/option.urdf.xacro (robot description, xacro)
@@ -29,3 +29,31 @@
     </link>
   </xacro:macro>
+  <xacro:macro name="lidar_multi_mount" params="prefix parent *joint_origin">
+    <joint name="${prefix}_joint" type="fixed">
+      <xacro:insert_block name="joint_origin" />
+      <parent link="${parent}" />
+      <child link="${prefix}_link" />
+    </joint>
+    <link name="${prefix}_link">
+      <visual>
+        <geometry>
+          <mesh filename="package://raspimouse_description/meshes/stl/RasPiMouse_MultiLiDARMount.stl" scale="0.001 0.001 0.001"/>
+        </geometry>
+      </visual>
+      <collision>
+        <!-- <geometry> -->
+          <!-- <mesh filename="package://raspimouse_description/meshes/stl/RasPiMouse_MultiLiDARMount.stl" scale="0.001 0.001 0.001"/> -->
+        <!-- </geometry> -->
+        <origin rpy="0 0 0" xyz="0.005 0 0.0435" />
+        <geometry>
+          <box size="0.117 0.080 0.087" />
+        </geometry>
+      </collision>
+      <inertial>
+        <origin xyz="0 0 0.07" />
+        <mass value="0.04"/>
+        <xacro:box_inertia m="0.04" x="0.13" y="0.1" z="0.002" />
+      </inertial>
+    </link>
+  </xacro:macro>
 </robot>

Commit message: Add colors

File: urdf/body/option.urdf.xacro (robot description, xacro)
@@ -40,4 +40,7 @@
           <mesh filename="package://raspimouse_description/meshes/stl/RasPiMouse_MultiLiDARMount.stl" scale="0.001 0.001 0.001"/>
         </geometry>
+        <material name="Light Black">
+          <color rgba="0.2 0.2 0.2 1.0" />
+        </material>
       </visual>
       <collision>

File: urdf/sensors/lidar.urdf.xacro (robot description, xacro)
@@ -42,4 +42,5 @@
           <mesh filename="package://raspimouse_description/meshes/stl/robotis-lds01.stl" scale="0.001 0.001 0.001"/>
         </geometry>
+        <material name="dark"/>
       </visual>
       <collision>

Commit message: Remove comment

File: urdf/body/option.urdf.xacro (robot description, xacro)
@@ -14,7 +14,4 @@
       </visual>
       <collision>
-        <!-- <geometry> -->
-          <!-- <mesh filename="package://raspimouse_description/meshes/dae/body/raspimouse_top_plate.dae"/> -->
-        <!-- </geometry> -->
         <origin rpy="0 0 0" xyz="0.005 0 0.0435" />
         <geometry>

Commit message: Adjusts the size of the collision of the multi_lidar_mount

File: urdf/body/option.urdf.xacro (robot description, xacro)
@@ -42,10 +42,7 @@
       </visual>
       <collision>
-        <!-- <geometry> -->
-          <!-- <mesh filename="package://raspimouse_description/meshes/stl/RasPiMouse_MultiLiDARMount.stl" scale="0.001 0.001 0.001"/> -->
-        <!-- </geometry> -->
-        <origin rpy="0 0 0" xyz="0.005 0 0.0435" />
+        <origin rpy="0 0 0" xyz="0.0 0 0.002" />
         <geometry>
-          <box size="0.117 0.080 0.087" />
+          <box size="0.135 0.095 0.005" />
         </geometry>
       </collision>

Commit message: Adjust the inertial position

File: urdf/body/option.urdf.xacro (robot description, xacro)
@@ -48,5 +48,5 @@
       </collision>
       <inertial>
-        <origin xyz="0 0 0.07" />
+        <origin xyz="0 0 0.0" />
         <mass value="0.04"/>
         <xacro:box_inertia m="0.04" x="0.13" y="0.1" z="0.002" />

Commit message: LiDARマウントの重心位置を修正

File: urdf/body/option.urdf.xacro (robot description, xacro)
@@ -48,5 +48,5 @@
       </collision>
       <inertial>
-        <origin xyz="0 0 0.0" />
+        <origin xyz="0 0 0.002" />
         <mass value="0.04"/>
         <xacro:box_inertia m="0.04" x="0.13" y="0.1" z="0.002" />

Commit message: LiDARの追加 (#38)
* Update descriptions

* Adds stl data of multi LIDAR mount

* Adds xacro if for lds and rplidar.

* Adds macro lidar_multi_mount

* Adds macro lidar_multi_sensor

* Update README. Adds License description

* Adds stl file for LDS

* Update specs

* Update collision size

* Adjust positions

* Add colors

* Adds legs for LDS

* fix typo

* Adds lidar parameter to macro lidar_multi_sensor.

* Adds RPLIDAR thing

* Adds lidar parameter to macro lidar_multi_sensor

* Adds if statement. rplidar is to be added

* Update README

* Update file name

* Update links

* Update lidar macro

* update macro names

* Adds RPLIDAR macros

* Update specs for RPLIDAR

* Updates the position of LDS and the length of its legs

* Updates RPLIDAR's position

* Adds a command that displays the lidar mounted on the robot.

* Replace material color to black

* Adds leg visual macro for the lidars

* Remove comments

* Update urdf/raspimouse.urdf.xacro

Co-authored-by: Shota Aoki <s.aoki@rt-net.jp>

* Adjust the collision size and position of the LIDARs

* Remove comment

* Adjusts the size of the collision of the multi_lidar_mount

* Adjust the inertial position

* Adjust the inertial height of each LIDAR

* LiDARマウントの重心位置を修正

Co-authored-by: Shota Aoki <s.aoki@rt-net.jp>

File: urdf/body/option.urdf.xacro (robot description, xacro)
@@ -14,7 +14,4 @@
       </visual>
       <collision>
-        <!-- <geometry> -->
-          <!-- <mesh filename="package://raspimouse_description/meshes/dae/body/raspimouse_top_plate.dae"/> -->
-        <!-- </geometry> -->
         <origin rpy="0 0 0" xyz="0.005 0 0.0435" />
         <geometry>
@@ -29,3 +26,31 @@
     </link>
   </xacro:macro>
+  <xacro:macro name="lidar_multi_mount" params="prefix parent *joint_origin">
+    <joint name="${prefix}_joint" type="fixed">
+      <xacro:insert_block name="joint_origin" />
+      <parent link="${parent}" />
+      <child link="${prefix}_link" />
+    </joint>
+    <link name="${prefix}_link">
+      <visual>
+        <geometry>
+          <mesh filename="package://raspimouse_description/meshes/stl/RasPiMouse_MultiLiDARMount.stl" scale="0.001 0.001 0.001"/>
+        </geometry>
+        <material name="Light Black">
+          <color rgba="0.2 0.2 0.2 1.0" />
+        </material>
+      </visual>
+      <collision>
+        <origin rpy="0 0 0" xyz="0.0 0 0.002" />
+        <geometry>
+          <box size="0.135 0.095 0.005" />
+        </geometry>
+      </collision>
+      <inertial>
+        <origin xyz="0 0 0.002" />
+        <mass value="0.04"/>
+        <xacro:box_inertia m="0.04" x="0.13" y="0.1" z="0.002" />
+      </inertial>
+    </link>
+  </xacro:macro>
 </robot>

File: urdf/raspimouse.urdf.xacro (robot description, xacro)
@@ -13,4 +13,7 @@
   <xacro:arg name="diffdrive_namespace" default="/" />
   <xacro:arg name="sensor_namespace" default="raspimouse_on_gazebo" />
+  <material name="black">
+    <color rgba="0.2 0.2 0.2 1.0"/>
+  </material>
   <xacro:include filename="$(find raspimouse_description)/urdf/common.xacro" />
   <xacro:include filename="$(find raspimouse_description)/urdf/body/body.urdf.xacro" />
@@ -61,4 +64,20 @@
     </xacro:lidar_urg_sensor>
   </xacro:if>
+  <xacro:if value="${'$(arg lidar)' == 'lds'}">
+    <xacro:lidar_multi_mount prefix="lds_multi_mount" parent="base_link">
+      <origin xyz="0 0 0.0855" rpy="0 0 0" />
+    </xacro:lidar_multi_mount>
+    <xacro:lidar_lds_sensor sensor_link_name="$(arg lidar_frame)" parent="$(arg lidar)_multi_mount_link">
+      <origin xyz="0.0 0.0 0.0345" rpy="0 0 3.14" />
+    </xacro:lidar_lds_sensor>
+  </xacro:if>
+  <xacro:if value="${'$(arg lidar)' == 'rplidar'}">
+    <xacro:lidar_multi_mount prefix="rplidar_multi_mount" parent="base_link">
+      <origin xyz="0 0 0.0855" rpy="0 0 0" />
+    </xacro:lidar_multi_mount>
+    <xacro:lidar_rp_sensor sensor_link_name="$(arg lidar_frame)" parent="$(arg lidar)_multi_mount_link">
+      <origin xyz="0.0 0.0 0.0445" rpy="0 0 3.14"/> <!-- The LIDAR is about 13cm from the ground-->
+    </xacro:lidar_rp_sensor>
+  </xacro:if>
   <!-- =============== Gazebo =============== -->
   <xacro:if value="$(arg gazebo_plugin)">
@@ -88,4 +107,10 @@
       <xacro:lidar_gazebo sensor_link_name="$(arg lidar_frame)" base_rad="0" rad_range="4.71" min_range="0.10" max_range="5.6" />
     </xacro:if>
+    <xacro:if value="${'$(arg lidar)' == 'lds'}">
+      <xacro:lidar_gazebo sensor_link_name="$(arg lidar_frame)" base_rad="0" rad_range="6.28" min_range="0.12" max_range="3.50" />
+    </xacro:if>
+    <xacro:if value="${'$(arg lidar)' == 'rplidar'}">
+      <xacro:lidar_gazebo sensor_link_name="$(arg lidar_frame)" base_rad="0" rad_range="6.28" min_range="0.15" max_range="12" />
+    </xacro:if>
     <!-- DiffDriveController -->
     <xacro:diffdrive_gazebo publish_tf="$(arg tf)" publish_jointstate="$(arg jointstate)"

File: urdf/sensors/lidar.urdf.xacro (robot description, xacro)
@@ -3,4 +3,34 @@
   <xacro:include filename="$(find raspimouse_description)/urdf/sensors/lidar.gazebo.xacro"/>
   <xacro:arg name="laser_visual" default="false"/>
+  <xacro:macro name="lidar_legs" params="length radius z_pos">
+    <visual>
+      <origin xyz="0.035 0.025 ${z_pos}" rpy="0 0 0" />
+      <geometry>
+        <cylinder length="${length}" radius="${radius}" />
+      </geometry>
+      <material name="black" />
+    </visual>
+    <visual>
+      <origin xyz="0.035 -0.025 ${z_pos}" rpy="0 0 0" />
+      <geometry>
+        <cylinder length="${length}" radius="${radius}" />
+      </geometry>
+      <material name="black" />
+    </visual>
+    <visual>
+      <origin xyz="-0.022 0.031 ${z_pos}" rpy="0 0 0" />
+      <geometry>
+        <cylinder length="${length}" radius="${radius}" />
+      </geometry>
+      <material name="black" />
+    </visual>
+    <visual>
+      <origin xyz="-0.022 -0.031 ${z_pos}" rpy="0 0 0" />
+      <geometry>
+        <cylinder length="${length}" radius="${radius}" />
+      </geometry>
+      <material name="black" />
+    </visual>
+  </xacro:macro>
   <xacro:macro name="lidar_urg_sensor" params="sensor_link_name parent *joint_origin">
     <joint name="${sensor_link_name}_joint" type="fixed">
@@ -16,7 +46,4 @@
       </visual>
       <collision>
-        <!-- <geometry> -->
-          <!-- <mesh filename="package://raspimouse_description/meshes/dae/sensor/urg_optical_axis_center_origin.dae"/> -->
-        <!-- </geometry> -->
         <origin xyz="0 0 -0.01815" />
         <geometry>
@@ -25,5 +52,5 @@
       </collision>
       <inertial>
-        <mass value="0.160" />
+        <mass value="0.16" />
         <origin xyz="0 0 0" />
         <xacro:cylinder_inertia m="0.16" r="0.025" h="0.07" />
@@ -31,3 +58,57 @@
     </link>
   </xacro:macro>
+  <xacro:macro name="lidar_lds_sensor" params="sensor_link_name parent *joint_origin">
+    <joint name="${sensor_link_name}_joint" type="fixed">
+      <xacro:insert_block name="joint_origin"/>
+      <parent link="${parent}"/>
+      <child link="${sensor_link_name}"/>
+    </joint>
+    <link name="${sensor_link_name}">
+      <visual>
+        <geometry>
+          <mesh filename="package://raspimouse_description/meshes/stl/robotis_lds01.stl" scale="0.001 0.001 0.001"/>
+        </geometry>
+        <material name="black"/>
+      </visual>
+      <xacro:lidar_legs length="0.019" radius="0.005" z_pos="-0.0228"/>
+      <collision>
+        <geometry>
+          <cylinder radius="0.035" length="0.040"/>
+        </geometry>
+        <origin xyz="0 0 -0.008" />
+      </collision>
+      <inertial>
+        <mass value="0.160" />
+        <origin xyz="0 0 0" />
+        <xacro:cylinder_inertia m="0.16" r="0.025" h="0.03" />
+      </inertial>
+    </link>
+  </xacro:macro>
+  <xacro:macro name="lidar_rp_sensor" params="sensor_link_name parent *joint_origin">
+    <joint name="${sensor_link_name}_joint" type="fixed">
+      <xacro:insert_block name="joint_origin"/>
+      <parent link="${parent}"/>
+      <child link="${sensor_link_name}"/>
+    </joint>
+    <link name="${sensor_link_name}">
+      <visual>
+        <geometry>
+          <mesh filename="package://raspimouse_description/meshes/stl/robotis_lds01.stl" scale="0.001 0.001 0.001"/>
+        </geometry>
+        <material name="black"/>
+      </visual>
+      <xacro:lidar_legs length="0.027" radius="0.003" z_pos="-0.028"/>
+      <collision>
+        <geometry>
+          <cylinder radius="0.036" length="0.042"/>
+        </geometry>
+        <origin xyz="0 0 -0.008" />
+      </collision>
+      <inertial>
+        <mass value="0.160" />
+        <origin xyz="0 0 0" />
+        <xacro:cylinder_inertia m="0.16" r="0.025" h="0.03" />
+      </inertial>
+    </link>
+  </xacro:macro>
 </robot>
