Commit message: Refactor

File: urdf/raspimouse.urdf (robot description, URDF)
Before this commit: robot raspimouse, 4 links, 3 joints
Links:
- removed link left_wheel
- removed link right_wheel
- added link left_wheel_link; visual mesh filename=package://raspimouse_description/meshes/dae/wheel/raspimous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
- added link right_wheel_link; visual mesh filename=package://raspimouse_description/meshes/dae/wheel/raspimous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
- link base_link: geometry visual mesh filename=package://raspimouse_description/meshes/dae/body/raspimouse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
Joints:
- joint left_wheel_joint: child left_wheel -> left_wheel_link
- joint right_wheel_joint: child right_wheel -> right_wheel_link

File: urdf/raspimouse.urdf.xacro (robot description, xacro)
@@ -41,14 +41,19 @@
   </xacro:wheel>
   <!-- Sensors -->
-  <xacro:light_sensor prefix="rf" parent="base_link">
+  <link name="lightsensors" />
+  <joint name="lightsensors_joint" type="fixed">
+    <parent link="base_link" />
+    <child link="lightsensors" />
+  </joint>
+  <xacro:light_sensor prefix="rf" parent="lightsensors">
     <origin xyz="0.04 -0.045 0.032" rpy="0 0 0" />
   </xacro:light_sensor>
-  <xacro:light_sensor prefix="rs" parent="base_link">
+  <xacro:light_sensor prefix="rs" parent="lightsensors">
     <origin xyz="0.059 -0.01 0.032" rpy="0 0 -1.04" />
   </xacro:light_sensor>
-  <xacro:light_sensor prefix="ls" parent="base_link">
+  <xacro:light_sensor prefix="ls" parent="lightsensors">
     <origin xyz="0.059 0.01 0.032" rpy="0 0 1.04" />
   </xacro:light_sensor>
-  <xacro:light_sensor prefix="lf" parent="base_link">
+  <xacro:light_sensor prefix="lf" parent="lightsensors">
     <origin xyz="0.04 0.045 0.032" rpy="0 0 0" />
   </xacro:light_sensor>

File: urdf/sensors/lightsens.gazebo.xacro (robot description, xacro)
@@ -2,5 +2,6 @@
 <robot xmlns:xacro="http://ros.org/wiki/xacro">
   <xacro:macro name="lightsensor_gazebo" params="prefix base_rad rad_range min_range max_range robotdescription_namespace robot_namespace">
-    <gazebo reference="${prefix}">
+    <gazebo reference="${prefix}_lightsensor_link">
+      <material>Gazebo/Gray</material>
       <sensor type="ray" name="${prefix}_lightsensor">
         <pose>0 0 0 0 0 0</pose>

File: urdf/sensors/lightsens.urdf.xacro (robot description, xacro)
@@ -7,13 +7,15 @@
       <xacro:insert_block name="joint_origin" />
       <parent link="${parent}" />
-      <child link="${prefix}" />
+      <child link="${prefix}_lightsensor_link" />
     </joint>
-    <link name="${prefix}">
+    <link name="${prefix}_lightsensor_link">
       <visual>
         <geometry>
           <box size="0.01 0.005 0.007" />
         </geometry>
+        <material name="Gray">
+          <color rgba="0.2 0.2 0.2 1" />
+        </material>
       </visual>
-      <material name="Gray" />
       <inertial>
         <mass value="0.000001" />
@@ -24,6 +26,4 @@
       </inertial>
     </link>
-    <!-- Set up laser gazebo details -->
-    <!-- <hokuyo_laser /> -->
   </xacro:macro>
 </robot>
