Commit message: Update urdf/common.xacro
Co-authored-by: Shota Aoki <s.aoki@rt-net.jp>

File: urdf/common.xacro (robot description, xacro)
@@ -7,5 +7,5 @@
   <!-- PROPERTY LIST -->
   <!-- All units in m-kg-s-radians unit system -->
-  <xacro:property name="M_PI" value="3.1415926535897931" />
+  <xacro:property name="M_PI" value="3.1415926535897932" />
   <!-- Inertial macros. Units are kg*m^2 -->
   <xacro:macro name="box_inertia" params="m x y z">

Commit message: Update urdf/common.xacro
Co-authored-by: Shota Aoki <s.aoki@rt-net.jp>

File: urdf/common.xacro (robot description, xacro)
@@ -20,7 +20,7 @@
   </xacro:macro>
   <xacro:macro name="sphere_inertia" params="m r">
-    <inertia ixx="${m*r*r/5}" ixy="0" ixz="0"
-             iyy="${m*r*r/5}" iyz="0"
-             izz="${m*r*r/5}" />
+    <inertia ixx="${m*r*r*2/5}" ixy="0" ixz="0"
+             iyy="${m*r*r*2/5}" iyz="0"
+             izz="${m*r*r*"/5}" />
   </xacro:macro>
 </robot>

Commit message: Update tread

File: urdf/common.xacro (robot description, xacro)
@@ -4,5 +4,5 @@
   <xacro:property name="wheel_length" value="0.010" />
   <xacro:property name="wheel_mass" value="0.0113" />
-  <xacro:property name="wheel_separation" value="0.0935" />
+  <xacro:property name="wheel_separation" value="0.095" />
   <!-- PROPERTY LIST -->
   <!-- All units in m-kg-s-radians unit system -->

Commit message: Update urdf/common.xacro
Co-authored-by: Shota Aoki <s.aoki@rt-net.jp>

File: urdf/common.xacro (robot description, xacro)
@@ -4,5 +4,5 @@
   <xacro:property name="wheel_length" value="0.010" />
   <xacro:property name="wheel_mass" value="0.0113" />
-  <xacro:property name="wheel_separation" value="0.095" />
+  <xacro:property name="wheel_separation" value="0.0925" />
   <!-- PROPERTY LIST -->
   <!-- All units in m-kg-s-radians unit system -->

Commit message: WHELL_VELOCITY_LIMITを設定

File: urdf/common.xacro (robot description, xacro)
@@ -8,4 +8,5 @@
   <!-- All units in m-kg-s-radians unit system -->
   <xacro:property name="M_PI" value="3.1415926535897932" />
+  <xacro:property name="WHEEL_VELOCITY_LIMIT" value="15" />
   <!-- Inertial macros. Units are kg*m^2 -->
   <xacro:macro name="box_inertia" params="m x y z">

File: urdf/wheel/diffdrive.gazebo_ros2_control.xacro (robot description, xacro)
@@ -1,4 +1,5 @@
 <?xml version="1.0"?>
 <robot xmlns:xacro="http://www.ros.org/wiki/xacro">
+  <xacro:include filename="$(find raspimouse_description)/urdf/common.xacro" />
   <xacro:macro name="diffdrive_gazebo_ros2_control_settings"
     params="name_hardware
@@ -11,6 +12,6 @@
       <joint name="${name_right_wheel_joint}">
         <command_interface name="velocity">
-          <param name="min">-1</param>
-          <param name="max">1</param>
+          <param name="min">-${WHEEL_VELOCITY_LIMIT}</param>
+          <param name="max">${WHEEL_VELOCITY_LIMIT}</param>
         </command_interface>
         <state_interface name="position"/>
@@ -20,6 +21,6 @@
       <joint name="${name_left_wheel_joint}">
         <command_interface name="velocity">
-          <param name="min">-1</param>
-          <param name="max">1</param>
+          <param name="min">-${WHEEL_VELOCITY_LIMIT}</param>
+          <param name="max">${WHEEL_VELOCITY_LIMIT}</param>
         </command_interface>
         <state_interface name="position"/>

Commit message: WHEEL_VELOCITY_LIMITを15から90に変更

File: urdf/common.xacro (robot description, xacro)
@@ -8,5 +8,5 @@
   <!-- All units in m-kg-s-radians unit system -->
   <xacro:property name="M_PI" value="3.1415926535897932" />
-  <xacro:property name="WHEEL_VELOCITY_LIMIT" value="15" />
+  <xacro:property name="WHEEL_VELOCITY_LIMIT" value="90" />
   <!-- Inertial macros. Units are kg*m^2 -->
   <xacro:macro name="box_inertia" params="m x y z">
