Commit message: Add laser link option

File: urdf/raspimouse.urdf.xacro (robot description, xacro)
@@ -6,4 +6,5 @@
        xmlns:xacro="http://ros.org/wiki/xacro">
   <xacro:arg name="lidar" default="none" />
+  <xacro:arg name="lidar_frame" default="laser" />
   <xacro:arg name="gazebo_plugin" default="false" />
   <xacro:arg name="tf" default="true" />
@@ -47,5 +48,5 @@
   </xacro:light_sensor>
   <xacro:if value="${'$(arg lidar)' == 'urg'}">
-    <xacro:lrf_sensor prefix="urg_lrf_link" parent="base_link">
+    <xacro:lrf_sensor prefix="urg_lrf_link" parent="base_link" laser_frame="$(arg lidar_frame)">
       <origin xyz="0.0 0.0 0.14060" rpy="0 0 0" />
     </xacro:lrf_sensor>

File: urdf/sensors/lrf.urdf.xacro (robot description, xacro)
@@ -2,5 +2,5 @@
 <robot name="urg_sensor" xmlns:xacro="http://ros.org/wiki/xacro">
   <xacro:include filename="$(find raspimouse_description)/urdf/sensors/lrf.gazebo.xacro"/>
-  <xacro:macro name="lrf_sensor" params="prefix parent *joint_origin">
+  <xacro:macro name="lrf_sensor" params="prefix parent laser_frame *joint_origin">
     <joint name="${prefix}_joint" type="fixed">
       <xacro:insert_block name="joint_origin"/>
@@ -30,4 +30,10 @@
       </inertial>
     </link>
+    <!-- tf virtual joint/link -->
+    <joint name="lidar_frame_joint" type="fixed">
+      <parent link="${prefix}" />
+      <child link="${laser_frame}" />
+    </joint>
+    <link name="${laser_frame}" />
   </xacro:macro>
 </robot>

Commit message: Define robotdescription namespace

File: urdf/raspimouse.urdf.xacro (robot description, xacro)
@@ -9,5 +9,5 @@
   <xacro:arg name="tf" default="true" />
   <xacro:arg name="jointstate" default="true" />
-  <xacro:arg name="robot_namespace" default="" />
+  <xacro:arg name="robot_namespace" default="/" />
   <xacro:arg name="diffdrive_namespace" default="/" />
   <xacro:arg name="sensor_namespace" default="raspimouse_on_gazebo" />
@@ -61,14 +61,18 @@
     <xacro:lightsensor_gazebo prefix="rf" base_rad="0"
       rad_range="0.3" min_range="0.01" max_range="0.6"
-      robot_namespace="$(arg sensor_namespace)" />
+      robot_namespace="$(arg sensor_namespace)"
+      robotdescription_namespace="$(arg robot_namespace)" />
     <xacro:lightsensor_gazebo prefix="rs" base_rad="-1.04"
       rad_range="0.3" min_range="0.01" max_range="0.6"
-      robot_namespace="$(arg sensor_namespace)" />
+      robot_namespace="$(arg sensor_namespace)"
+      robotdescription_namespace="$(arg robot_namespace)" />
     <xacro:lightsensor_gazebo prefix="ls" base_rad="1.04"
       rad_range="0.3" min_range="0.01" max_range="0.6"
-      robot_namespace="$(arg sensor_namespace)" />
+      robot_namespace="$(arg sensor_namespace)"
+      robotdescription_namespace="$(arg robot_namespace)" />
     <xacro:lightsensor_gazebo prefix="lf" base_rad="0"
       rad_range="0.3" min_range="0.01" max_range="0.6"
-      robot_namespace="$(arg sensor_namespace)" />
+      robot_namespace="$(arg sensor_namespace)"
+      robotdescription_namespace="$(arg robot_namespace)" />
     <xacro:if value="${'$(arg lidar)' == 'urg'}">
       <xacro:lrf_gazebo prefix="urg" base_rad="0" rad_range="4.71" min_range="0.10" max_range="5.6" />

File: urdf/sensors/lightsens.gazebo.xacro (robot description, xacro)
@@ -1,5 +1,5 @@
 <?xml version="1.0"?>
 <robot xmlns:xacro="http://ros.org/wiki/xacro">
-  <xacro:macro name="lightsensor_gazebo" params="prefix base_rad rad_range min_range max_range robot_namespace">
+  <xacro:macro name="lightsensor_gazebo" params="prefix base_rad rad_range min_range max_range robotdescription_namespace robot_namespace">
     <gazebo reference="${prefix}">
       <sensor type="ray" name="${prefix}_lightsensor">
@@ -30,5 +30,5 @@
           <robotNamespace>${robot_namespace}</robotNamespace>
           <topicName>${prefix}_scan</topicName>
-          <frameName>${prefix}</frameName>
+          <frameName>${robotdescription_namespace}${prefix}</frameName>
         </plugin>
       </sensor>

Commit message: s/laser_frame/lidar_frame/g

File: urdf/raspimouse.urdf.xacro (robot description, xacro)
@@ -48,5 +48,5 @@
   </xacro:light_sensor>
   <xacro:if value="${'$(arg lidar)' == 'urg'}">
-    <xacro:lrf_sensor prefix="urg_lrf_link" parent="base_link" laser_frame="$(arg lidar_frame)">
+    <xacro:lrf_sensor prefix="urg_lrf_link" parent="base_link" lidar_frame="$(arg lidar_frame)">
       <origin xyz="0.0 0.0 0.14060" rpy="0 0 0" />
     </xacro:lrf_sensor>

File: urdf/sensors/lrf.urdf.xacro (robot description, xacro)
@@ -2,5 +2,5 @@
 <robot name="urg_sensor" xmlns:xacro="http://ros.org/wiki/xacro">
   <xacro:include filename="$(find raspimouse_description)/urdf/sensors/lrf.gazebo.xacro"/>
-  <xacro:macro name="lrf_sensor" params="prefix parent laser_frame *joint_origin">
+  <xacro:macro name="lrf_sensor" params="prefix parent lidar_frame *joint_origin">
     <joint name="${prefix}_joint" type="fixed">
       <xacro:insert_block name="joint_origin"/>
@@ -33,7 +33,7 @@
     <joint name="lidar_frame_joint" type="fixed">
       <parent link="${prefix}" />
-      <child link="${laser_frame}" />
+      <child link="${lidar_frame}" />
     </joint>
-    <link name="${laser_frame}" />
+    <link name="${lidar_frame}" />
   </xacro:macro>
 </robot>

Commit message: Update lidar_frame name option

File: urdf/raspimouse.urdf.xacro (robot description, xacro)
@@ -18,5 +18,5 @@
   <xacro:include filename="$(find raspimouse_description)/urdf/wheel/diffdrive.gazebo.xacro" />
   <xacro:include filename="$(find raspimouse_description)/urdf/sensors/lightsens.urdf.xacro" />
-  <xacro:include filename="$(find raspimouse_description)/urdf/sensors/lrf.urdf.xacro" />
+  <xacro:include filename="$(find raspimouse_description)/urdf/sensors/lidar.urdf.xacro" />
   <!-- =============== Link & Joint =============== -->
   <!-- Base -->
@@ -48,7 +48,7 @@
   </xacro:light_sensor>
   <xacro:if value="${'$(arg lidar)' == 'urg'}">
-    <xacro:lrf_sensor prefix="urg_lrf_link" parent="base_link" lidar_frame="$(arg lidar_frame)">
+    <xacro:lidar_urg_sensor sensor_link_name="$(arg lidar_frame)" parent="base_link">
       <origin xyz="0.0 0.0 0.14060" rpy="0 0 0" />
-    </xacro:lrf_sensor>
+    </xacro:lidar_urg_sensor>
   </xacro:if>
   <!-- =============== Gazebo =============== -->
@@ -77,5 +77,5 @@
       robotdescription_namespace="$(arg robot_namespace)" />
     <xacro:if value="${'$(arg lidar)' == 'urg'}">
-      <xacro:lrf_gazebo prefix="urg" base_rad="0" rad_range="4.71" min_range="0.10" max_range="5.6" />
+      <xacro:lidar_gazebo sensor_link_name="$(arg lidar_frame)" base_rad="0" rad_range="4.71" min_range="0.10" max_range="5.6" />
     </xacro:if>
     <!-- DiffDriveController -->

File: urdf/sensors/lidar.gazebo.xacro (robot description, xacro)
@@ -1,9 +1,8 @@
 <?xml version="1.0"?>
 <robot xmlns:xacro="http://ros.org/wiki/xacro">
-  <xacro:macro name="lrf_gazebo" params="prefix base_rad rad_range min_range max_range">
-    <gazebo reference="${prefix}_lrf_link">
-      <sensor type="ray" name="${prefix}_lrf_sensor">
-        <!-- <pose>0.0 0.0 0.05315 0 0 0</pose> -->
-        <pose>0 0 1 0 0 0</pose>
+  <xacro:macro name="lidar_gazebo" params="sensor_link_name base_rad rad_range min_range max_range">
+    <gazebo reference="${sensor_link_name}">
+      <sensor type="ray" name="${sensor_link_name}_sensor">
+        <pose>0 0 0 0 0 0</pose>
         <visualize>false</visualize>
         <update_rate>10</update_rate>
@@ -28,7 +27,7 @@
           </noise>
         </ray>
-        <plugin name="gazebo_ros_${prefix}_lrf_controller" filename="libgazebo_ros_laser.so">
+        <plugin name="gazebo_ros_${sensor_link_name}_controller" filename="libgazebo_ros_laser.so">
           <topicName>scan</topicName>
-          <frameName>${prefix}_lrf_link</frameName>
+          <frameName>${sensor_link_name}</frameName>
         </plugin>
       </sensor>

File: urdf/sensors/lidar.urdf.xacro (robot description, xacro)
@@ -1,12 +1,12 @@
 <?xml version="1.0"?>
 <robot name="urg_sensor" xmlns:xacro="http://ros.org/wiki/xacro">
-  <xacro:include filename="$(find raspimouse_description)/urdf/sensors/lrf.gazebo.xacro"/>
-  <xacro:macro name="lrf_sensor" params="prefix parent lidar_frame *joint_origin">
-    <joint name="${prefix}_joint" type="fixed">
+  <xacro:include filename="$(find raspimouse_description)/urdf/sensors/lidar.gazebo.xacro"/>
+  <xacro:macro name="lidar_urg_sensor" params="sensor_link_name parent *joint_origin">
+    <joint name="${sensor_link_name}_joint" type="fixed">
       <xacro:insert_block name="joint_origin"/>
       <parent link="${parent}"/>
-      <child link="${prefix}"/>
+      <child link="${sensor_link_name}"/>
     </joint>
-    <link name="${prefix}">
+    <link name="${sensor_link_name}">
       <visual>
         <geometry>
@@ -26,14 +26,7 @@
         <mass value="0.160" />
         <origin xyz="0 0 0" />
-        <inertia ixx="0.0001" ixy="0.0" ixz="0.0"
-          iyy="0.0001" iyz="0.0" izz="0.0001" />
+        <xacro:cylinder_inertia m="0.16" r="0.025" h="0.07" />
       </inertial>
     </link>
-    <!-- tf virtual joint/link -->
-    <joint name="lidar_frame_joint" type="fixed">
-      <parent link="${prefix}" />
-      <child link="${lidar_frame}" />
-    </joint>
-    <link name="${lidar_frame}" />
   </xacro:macro>
 </robot>

Commit message: Make lidar_frame name variable

File: urdf/raspimouse.urdf.xacro (robot description, xacro)
@@ -6,4 +6,6 @@
        xmlns:xacro="http://ros.org/wiki/xacro">
   <xacro:arg name="lidar" default="none" />
+  <xacro:arg name="lidar_frame" default="laser" />
+  <xacro:arg name="laser_visual" default="true"/>
   <xacro:arg name="gazebo_plugin" default="false" />
   <xacro:arg name="tf" default="true" />
@@ -17,5 +19,5 @@
   <xacro:include filename="$(find raspimouse_description)/urdf/wheel/diffdrive.gazebo.xacro" />
   <xacro:include filename="$(find raspimouse_description)/urdf/sensors/lightsens.urdf.xacro" />
-  <xacro:include filename="$(find raspimouse_description)/urdf/sensors/lrf.urdf.xacro" />
+  <xacro:include filename="$(find raspimouse_description)/urdf/sensors/lidar.urdf.xacro" />
   <!-- =============== Link & Joint =============== -->
   <!-- Base -->
@@ -47,7 +49,7 @@
   </xacro:light_sensor>
   <xacro:if value="${'$(arg lidar)' == 'urg'}">
-    <xacro:lrf_sensor prefix="urg_lrf_link" parent="base_link">
+    <xacro:lidar_urg_sensor sensor_link_name="$(arg lidar_frame)" parent="base_link">
       <origin xyz="0.0 0.0 0.14060" rpy="0 0 0" />
-    </xacro:lrf_sensor>
+    </xacro:lidar_urg_sensor>
   </xacro:if>
   <!-- =============== Gazebo =============== -->
@@ -76,5 +78,5 @@
       robotdescription_namespace="$(arg robot_namespace)" />
     <xacro:if value="${'$(arg lidar)' == 'urg'}">
-      <xacro:lrf_gazebo prefix="urg" base_rad="0" rad_range="4.71" min_range="0.10" max_range="5.6" />
+      <xacro:lidar_gazebo sensor_link_name="$(arg lidar_frame)" base_rad="0" rad_range="4.71" min_range="0.10" max_range="5.6" />
     </xacro:if>
     <!-- DiffDriveController -->

File: urdf/sensors/lidar.gazebo.xacro (robot description, xacro)
@@ -1,7 +1,7 @@
 <?xml version="1.0"?>
 <robot xmlns:xacro="http://ros.org/wiki/xacro">
-  <xacro:macro name="lrf_gazebo" params="prefix base_rad rad_range min_range max_range">
-    <gazebo reference="${prefix}_lrf_link">
-      <sensor type="ray" name="${prefix}_lrf_sensor">
+  <xacro:macro name="lidar_gazebo" params="sensor_link_name base_rad rad_range min_range max_range">
+    <gazebo reference="${sensor_link_name}">
+      <sensor type="ray" name="${sensor_link_name}_sensor">
         <pose>0 0 0 0 0 0</pose>
         <visualize>$(arg laser_visual)</visualize>
@@ -27,7 +27,7 @@
           </noise>
         </ray>
-        <plugin name="gazebo_ros_${prefix}_lrf_controller" filename="libgazebo_ros_laser.so">
+        <plugin name="gazebo_ros_${sensor_link_name}_controller" filename="libgazebo_ros_laser.so">
           <topicName>scan</topicName>
-          <frameName>${prefix}_lrf_link</frameName>
+          <frameName>${sensor_link_name}</frameName>
         </plugin>
       </sensor>

File: urdf/sensors/lidar.urdf.xacro (robot description, xacro)
@@ -1,13 +1,12 @@
 <?xml version="1.0"?>
 <robot name="urg_sensor" xmlns:xacro="http://ros.org/wiki/xacro">
-  <xacro:include filename="$(find raspimouse_description)/urdf/sensors/lrf.gazebo.xacro"/>
-  <xacro:arg name="laser_visual" default="false"/>
-  <xacro:macro name="lrf_sensor" params="prefix parent *joint_origin">
-    <joint name="${prefix}_joint" type="fixed">
+  <xacro:include filename="$(find raspimouse_description)/urdf/sensors/lidar.gazebo.xacro"/>
+  <xacro:macro name="lidar_urg_sensor" params="sensor_link_name parent *joint_origin">
+    <joint name="${sensor_link_name}_joint" type="fixed">
       <xacro:insert_block name="joint_origin"/>
       <parent link="${parent}"/>
-      <child link="${prefix}"/>
+      <child link="${sensor_link_name}"/>
     </joint>
-    <link name="${prefix}">
+    <link name="${sensor_link_name}">
       <visual>
         <geometry>
@@ -27,6 +26,5 @@
         <mass value="0.160" />
         <origin xyz="0 0 0" />
-        <inertia ixx="0.0001" ixy="0.0" ixz="0.0"
-          iyy="0.0001" iyz="0.0" izz="0.0001" />
+        <xacro:cylinder_inertia m="0.16" r="0.025" h="0.07" />
       </inertial>
     </link>

Commit message: Refactor

File: urdf/raspimouse.urdf.xacro (robot description, xacro)
@@ -36,14 +36,19 @@
   </xacro:wheel>
   <!-- Sensors -->
-  <xacro:light_sensor prefix="rf" parent="base_link">
+  <link name="lightsensors" />
+  <joint name="lightsensors_joint" type="fixed">
+    <parent link="base_link" />
+    <child link="lightsensors" />
+  </joint>
+  <xacro:light_sensor prefix="rf" parent="lightsensors">
     <origin xyz="0.04 -0.045 0.032" rpy="0 0 0" />
   </xacro:light_sensor>
-  <xacro:light_sensor prefix="rs" parent="base_link">
+  <xacro:light_sensor prefix="rs" parent="lightsensors">
     <origin xyz="0.059 -0.01 0.032" rpy="0 0 -1.04" />
   </xacro:light_sensor>
-  <xacro:light_sensor prefix="ls" parent="base_link">
+  <xacro:light_sensor prefix="ls" parent="lightsensors">
     <origin xyz="0.059 0.01 0.032" rpy="0 0 1.04" />
   </xacro:light_sensor>
-  <xacro:light_sensor prefix="lf" parent="base_link">
+  <xacro:light_sensor prefix="lf" parent="lightsensors">
     <origin xyz="0.04 0.045 0.032" rpy="0 0 0" />
   </xacro:light_sensor>

Commit message: Add lidar link rename option (#23)
* Fix wheel link missing problem

Also, add comments about params

-wheelTorque: 5
+wheelTorque: 500

Co-authored-by: Shota Aoki <s.aoki@rt-net.jp>

* Fix typo to suppress warnings loading GazeboPlugin

same as https://github.com/rt-net/jnmouse_description/pull/9

* Fix default namespace to avoid odometry tf error

related: https://github.com/rt-net/raspimouse_sim/pull/55

* Refactor

* Add an option to load gazebo plugin to allow URDF to be loaded without gazebo_ros

* Separate DiffDriveController into separate files

* Add laser link option

* s/laser_frame/lidar_frame/g

* Update lidar_frame name option

Co-authored-by: Shota Aoki <s.aoki@rt-net.jp>

File: urdf/raspimouse.urdf.xacro (robot description, xacro)
@@ -6,4 +6,5 @@
        xmlns:xacro="http://ros.org/wiki/xacro">
   <xacro:arg name="lidar" default="none" />
+  <xacro:arg name="lidar_frame" default="laser" />
   <xacro:arg name="gazebo_plugin" default="false" />
   <xacro:arg name="tf" default="true" />
@@ -17,5 +18,5 @@
   <xacro:include filename="$(find raspimouse_description)/urdf/wheel/diffdrive.gazebo.xacro" />
   <xacro:include filename="$(find raspimouse_description)/urdf/sensors/lightsens.urdf.xacro" />
-  <xacro:include filename="$(find raspimouse_description)/urdf/sensors/lrf.urdf.xacro" />
+  <xacro:include filename="$(find raspimouse_description)/urdf/sensors/lidar.urdf.xacro" />
   <!-- =============== Link & Joint =============== -->
   <!-- Base -->
@@ -47,7 +48,7 @@
   </xacro:light_sensor>
   <xacro:if value="${'$(arg lidar)' == 'urg'}">
-    <xacro:lrf_sensor prefix="urg_lrf_link" parent="base_link">
+    <xacro:lidar_urg_sensor sensor_link_name="$(arg lidar_frame)" parent="base_link">
       <origin xyz="0.0 0.0 0.14060" rpy="0 0 0" />
-    </xacro:lrf_sensor>
+    </xacro:lidar_urg_sensor>
   </xacro:if>
   <!-- =============== Gazebo =============== -->
@@ -76,5 +77,5 @@
       robotdescription_namespace="$(arg robot_namespace)" />
     <xacro:if value="${'$(arg lidar)' == 'urg'}">
-      <xacro:lrf_gazebo prefix="urg" base_rad="0" rad_range="4.71" min_range="0.10" max_range="5.6" />
+      <xacro:lidar_gazebo sensor_link_name="$(arg lidar_frame)" base_rad="0" rad_range="4.71" min_range="0.10" max_range="5.6" />
     </xacro:if>
     <!-- DiffDriveController -->

File: urdf/sensors/lidar.urdf.xacro (robot description, xacro)
@@ -1,12 +1,12 @@
 <?xml version="1.0"?>
 <robot name="urg_sensor" xmlns:xacro="http://ros.org/wiki/xacro">
-  <xacro:include filename="$(find raspimouse_description)/urdf/sensors/lrf.gazebo.xacro"/>
-  <xacro:macro name="lrf_sensor" params="prefix parent *joint_origin">
-    <joint name="${prefix}_joint" type="fixed">
+  <xacro:include filename="$(find raspimouse_description)/urdf/sensors/lidar.gazebo.xacro"/>
+  <xacro:macro name="lidar_urg_sensor" params="sensor_link_name parent *joint_origin">
+    <joint name="${sensor_link_name}_joint" type="fixed">
       <xacro:insert_block name="joint_origin"/>
       <parent link="${parent}"/>
-      <child link="${prefix}"/>
+      <child link="${sensor_link_name}"/>
     </joint>
-    <link name="${prefix}">
+    <link name="${sensor_link_name}">
       <visual>
         <geometry>
@@ -26,6 +26,5 @@
         <mass value="0.160" />
         <origin xyz="0 0 0" />
-        <inertia ixx="0.0001" ixy="0.0" ixz="0.0"
-          iyy="0.0001" iyz="0.0" izz="0.0001" />
+        <xacro:cylinder_inertia m="0.16" r="0.025" h="0.07" />
       </inertial>
     </link>

Commit message: Adds xacro if for lds and rplidar.

File: urdf/raspimouse.urdf.xacro (robot description, xacro)
@@ -61,4 +61,12 @@
     </xacro:lidar_urg_sensor>
   </xacro:if>
+  <xacro:if value="${'$(arg lidar)' == 'lds'}">
+    <xacro:lidar_multi_mount prefix="lds_multi_mount" parent="base_link">
+      <origin xyz="0 0 0" rpy="0 0 0" />
+    </xacro:lidar_multi_mount>
+    <xacro:lidar_multi_sensor sensor_link_name="$(arg lidar_frame)" parent="lds_multi_mount_link">
+      <origin xyz="0.0 0.0 0.0" rpy="0 0 0" />
+    </xacro:lidar_multi_sensor>
+  </xacro:if>
   <!-- =============== Gazebo =============== -->
   <xacro:if value="$(arg gazebo_plugin)">
@@ -88,4 +96,10 @@
       <xacro:lidar_gazebo sensor_link_name="$(arg lidar_frame)" base_rad="0" rad_range="4.71" min_range="0.10" max_range="5.6" />
     </xacro:if>
+    <xacro:if value="${'$(arg lidar)' == 'lds'}">
+      <xacro:lidar_gazebo sensor_link_name="$(arg lidar_frame)" base_rad="0" rad_range="4.71" min_range="0.10" max_range="5.6" />
+    </xacro:if>
+    <xacro:if value="${'$(arg lidar)' == 'rplidar'}">
+      <xacro:lidar_gazebo sensor_link_name="$(arg lidar_frame)" base_rad="0" rad_range="4.71" min_range="0.10" max_range="5.6" />
+    </xacro:if>
     <!-- DiffDriveController -->
     <xacro:diffdrive_gazebo publish_tf="$(arg tf)" publish_jointstate="$(arg jointstate)"

Commit message: Adjust positions

File: urdf/raspimouse.urdf.xacro (robot description, xacro)
@@ -63,8 +63,8 @@
   <xacro:if value="${'$(arg lidar)' == 'lds'}">
     <xacro:lidar_multi_mount prefix="lds_multi_mount" parent="base_link">
-      <origin xyz="0 0 0" rpy="0 0 0" />
+      <origin xyz="0 0 0.0855" rpy="0 0 0" />
     </xacro:lidar_multi_mount>
     <xacro:lidar_multi_sensor sensor_link_name="$(arg lidar_frame)" parent="lds_multi_mount_link">
-      <origin xyz="0.0 0.0 0.0" rpy="0 0 0" />
+      <origin xyz="0.0 0.0 0.035" rpy="0 0 3.14" />
     </xacro:lidar_multi_sensor>
   </xacro:if>

Commit message: Adds RPLIDAR thing

File: urdf/raspimouse.urdf.xacro (robot description, xacro)
@@ -69,4 +69,11 @@
     </xacro:lidar_multi_sensor>
   </xacro:if>
+  <xacro:if value="${'$(arg lidar)' == 'rplidar'}">
+    <xacro:lidar_multi_mount prefix="rplidar_multi_mount" parent="base_link">
+      <origin xyz="0 0 0.0855" rpy="0 0 0" />
+    </xacro:lidar_multi_mount>
+    <xacro:lidar_multi_sensor sensor_link_name="$(arg lidar_frame)" parent="$(arg lidar)_multi_mount_link" lidar="$(arg lidar)">
+    </xacro:lidar_multi_sensor>
+  </xacro:if>
   <!-- =============== Gazebo =============== -->
   <xacro:if value="$(arg gazebo_plugin)">

Commit message: Update specs for RPLIDAR

File: urdf/raspimouse.urdf.xacro (robot description, xacro)
@@ -107,5 +107,5 @@
     </xacro:if>
     <xacro:if value="${'$(arg lidar)' == 'rplidar'}">
-      <xacro:lidar_gazebo sensor_link_name="$(arg lidar_frame)" base_rad="0" rad_range="4.71" min_range="0.10" max_range="5.6" />
+      <xacro:lidar_gazebo sensor_link_name="$(arg lidar_frame)" base_rad="0" rad_range="6.28" min_range="0.15" max_range="10" />
     </xacro:if>
     <!-- DiffDriveController -->

File: urdf/sensors/lidar.urdf.xacro (robot description, xacro)
@@ -136,5 +136,5 @@
         <!-- </geometry> -->
         <geometry>
-          <cylinder radius="0.035" length="0.040"/>
+          <cylinder radius="0.048" length="0.055"/>
         </geometry>
         <origin xyz="0 0 -0.01815" />

Commit message: Updates the position of LDS and the length of its legs

File: urdf/raspimouse.urdf.xacro (robot description, xacro)
@@ -66,5 +66,5 @@
     </xacro:lidar_multi_mount>
     <xacro:lidar_lds_sensor sensor_link_name="$(arg lidar_frame)" parent="$(arg lidar)_multi_mount_link">
-      <origin xyz="0.0 0.0 0.035" rpy="0 0 3.14" />
+      <origin xyz="0.0 0.0 0.0345" rpy="0 0 3.14" />
     </xacro:lidar_lds_sensor>
   </xacro:if>

File: urdf/sensors/lidar.urdf.xacro (robot description, xacro)
@@ -48,5 +48,5 @@
         <origin xyz="0.035 0.025 -0.0228" rpy="0 0 0" />
         <geometry>
-          <cylinder length="0.02" radius="0.005" />
+          <cylinder length="0.019" radius="0.005" />
         </geometry>
         <material name="dark" />
@@ -55,5 +55,5 @@
         <origin xyz="0.035 -0.025 -0.0228" rpy="0 0 0" />
         <geometry>
-          <cylinder length="0.02" radius="0.005" />
+          <cylinder length="0.019" radius="0.005" />
         </geometry>
         <material name="dark" />
@@ -62,5 +62,5 @@
         <origin xyz="-0.022 0.031 -0.0228" rpy="0 0 0" />
         <geometry>
-          <cylinder length="0.02" radius="0.005" />
+          <cylinder length="0.019" radius="0.005" />
         </geometry>
         <material name="dark" />
@@ -69,5 +69,5 @@
         <origin xyz="-0.022 -0.031 -0.0228" rpy="0 0 0" />
         <geometry>
-          <cylinder length="0.02" radius="0.005" />
+          <cylinder length="0.019" radius="0.005" />
         </geometry>
         <material name="dark" />
