Commit message: Updates RPLIDAR's position

File: urdf/raspimouse.urdf.xacro (robot description, xacro)
@@ -74,4 +74,5 @@
     </xacro:lidar_multi_mount>
     <xacro:lidar_rp_sensor sensor_link_name="$(arg lidar_frame)" parent="$(arg lidar)_multi_mount_link">
+      <origin xyz="0.0 0.0 0.0445" rpy="0 0 3.14"/> <!-- The LIDAR is about 13cm from the ground-->
     </xacro:lidar_rp_sensor>
   </xacro:if>

File: urdf/sensors/lidar.urdf.xacro (robot description, xacro)
@@ -104,28 +104,28 @@
       <!-- Legs -->
       <visual>
-        <origin xyz="0.035 0.025 -0.0228" rpy="0 0 0" />
+        <origin xyz="0.035 0.025 -0.028" rpy="0 0 0" />
         <geometry>
-          <cylinder length="0.02" radius="0.005" />
+          <cylinder length="0.027" radius="0.003" />
         </geometry>
         <material name="dark" />
       </visual>
       <visual>
-        <origin xyz="0.035 -0.025 -0.0228" rpy="0 0 0" />
+        <origin xyz="0.035 -0.025 -0.028" rpy="0 0 0" />
         <geometry>
-          <cylinder length="0.02" radius="0.005" />
+          <cylinder length="0.027" radius="0.003" />
         </geometry>
         <material name="dark" />
       </visual>
       <visual>
-        <origin xyz="-0.022 0.031 -0.0228" rpy="0 0 0" />
+        <origin xyz="-0.022 0.031 -0.028" rpy="0 0 0" />
         <geometry>
-          <cylinder length="0.02" radius="0.005" />
+          <cylinder length="0.027" radius="0.003" />
         </geometry>
         <material name="dark" />
       </visual>
       <visual>
-        <origin xyz="-0.022 -0.031 -0.0228" rpy="0 0 0" />
+        <origin xyz="-0.022 -0.031 -0.028" rpy="0 0 0" />
         <geometry>
-          <cylinder length="0.02" radius="0.005" />
+          <cylinder length="0.027" radius="0.003" />
         </geometry>
         <material name="dark" />

Commit message: Replace material color to black

File: urdf/raspimouse.urdf.xacro (robot description, xacro)
@@ -13,4 +13,7 @@
   <xacro:arg name="diffdrive_namespace" default="/" />
   <xacro:arg name="sensor_namespace" default="raspimouse_on_gazebo" />
+  <material name="black">
+    <color rgba="0.2 0.2 0.2 1.0"/>
+  </material>
   <xacro:include filename="$(find raspimouse_description)/urdf/common.xacro" />
   <xacro:include filename="$(find raspimouse_description)/urdf/body/body.urdf.xacro" />

File: urdf/sensors/lidar.urdf.xacro (robot description, xacro)
@@ -25,5 +25,5 @@
       </collision>
       <inertial>
-        <mass value="0.160" />
+        <mass value="0.16" />
         <origin xyz="0 0 0" />
         <xacro:cylinder_inertia m="0.16" r="0.025" h="0.07" />
@@ -42,5 +42,5 @@
           <mesh filename="package://raspimouse_description/meshes/stl/robotis_lds01.stl" scale="0.001 0.001 0.001"/>
         </geometry>
-        <material name="dark"/>
+        <material name="black"/>
       </visual>
       <!-- Legs -->
@@ -50,5 +50,5 @@
           <cylinder length="0.019" radius="0.005" />
         </geometry>
-        <material name="dark" />
+        <material name="black" />
       </visual>
       <visual>
@@ -57,5 +57,5 @@
           <cylinder length="0.019" radius="0.005" />
         </geometry>
-        <material name="dark" />
+        <material name="black" />
       </visual>
       <visual>
@@ -64,5 +64,5 @@
           <cylinder length="0.019" radius="0.005" />
         </geometry>
-        <material name="dark" />
+        <material name="black" />
       </visual>
       <visual>
@@ -71,5 +71,5 @@
           <cylinder length="0.019" radius="0.005" />
         </geometry>
-        <material name="dark" />
+        <material name="black" />
       </visual>
       <collision>
@@ -100,5 +100,5 @@
           <mesh filename="package://raspimouse_description/meshes/stl/robotis_lds01.stl" scale="0.001 0.001 0.001"/>
         </geometry>
-        <material name="dark"/>
+        <material name="black"/>
       </visual>
       <!-- Legs -->
@@ -108,5 +108,5 @@
           <cylinder length="0.027" radius="0.003" />
         </geometry>
-        <material name="dark" />
+        <material name="black" />
       </visual>
       <visual>
@@ -115,5 +115,5 @@
           <cylinder length="0.027" radius="0.003" />
         </geometry>
-        <material name="dark" />
+        <material name="black" />
       </visual>
       <visual>
@@ -122,5 +122,5 @@
           <cylinder length="0.027" radius="0.003" />
         </geometry>
-        <material name="dark" />
+        <material name="black" />
       </visual>
       <visual>
@@ -129,5 +129,5 @@
           <cylinder length="0.027" radius="0.003" />
         </geometry>
-        <material name="dark" />
+        <material name="black" />
       </visual>
       <collision>

Commit message: controller_managerを起動するように変更

File: urdf/raspimouse.urdf.xacro (robot description, xacro)
@@ -13,4 +13,7 @@
   <xacro:arg name="diffdrive_namespace" default="/" />
   <xacro:arg name="sensor_namespace" default="raspimouse_on_gazebo" />
+  <xacro:arg name="use_gazebo" default="false" />
+  <xacro:arg name="gz_control_config_package" default="" />
+  <xacro:arg name="gz_control_config_file_path" default="" />
   <material name="black">
     <color rgba="0.2 0.2 0.2 1.0"/>
@@ -21,4 +24,5 @@
   <xacro:include filename="$(find raspimouse_description)/urdf/wheel/wheel.urdf.xacro" />
   <xacro:include filename="$(find raspimouse_description)/urdf/wheel/diffdrive.gazebo.xacro" />
+  <xacro:include filename="$(find raspimouse_description)/urdf/wheel/diffdrive.gazebo_ros2_control.xacro" />
   <xacro:include filename="$(find raspimouse_description)/urdf/sensors/lightsens.urdf.xacro" />
   <xacro:include filename="$(find raspimouse_description)/urdf/sensors/lidar.urdf.xacro" />
@@ -81,4 +85,20 @@
   </xacro:if>
   <!-- =============== Gazebo =============== -->
+  <xacro:if value="$(arg use_gazebo)">
+    <xacro:gazebo_robot_settings
+      name_hardware="GazeboSystem"
+      name_right_wheel_joint="right_wheel_joint"
+      name_left_wheel_joint="left_wheel_joint"
+      use_gazebo="$(arg use_gazebo)"
+      config_file_package="$(arg gz_control_config_package)"
+      config_file_path="$(arg gz_control_config_file_path)" />
+    <xacro:raspimouse_gazebo_ros2_control_settings
+      name_hardware="GazeboSystem"
+      name_right_wheel_joint="right_wheel_joint"
+      name_left_wheel_joint="left_wheel_joint"
+      use_gazebo="$(arg use_gazebo)"
+      config_file_package="$(arg gz_control_config_package)"
+      config_file_path="$(arg gz_control_config_file_path)" />
+  </xacro:if>
   <xacro:if value="$(arg gazebo_plugin)">
     <gazebo>

File: urdf/wheel/diffdrive.gazebo.xacro (robot description, xacro)
@@ -2,4 +2,26 @@
 <robot name="diffdrive_gazebo" xmlns:xacro="http://ros.org/wiki/xacro">
   <xacro:include filename="$(find raspimouse_description)/urdf/common.xacro" />
+  <xacro:macro name="gazebo_robot_settings"
+    params="name_hardware
+            name_right_wheel_joint
+            name_left_wheel_joint
+            use_gazebo
+            config_file_package
+            config_file_path
+            ">
+    <gazebo>
+      <xacro:if value="${use_gazebo}">
+        <plugin filename="libign_ros2_control-system.so" name="ign_ros2_control::IgnitionROS2ControlPlugin">
+          <parameters>$(find ${config_file_package})/${config_file_path}</parameters>
+        </plugin>
+      </xacro:if>
+      <xacro:unless value="${use_gazebo}">
+        <plugin filename="libgazebo_ros2_control.so" name="gazebo_ros2_control">
+          <robot_sim_type>gazebo_ros2_control/GazeboSystem</robot_sim_type>
+          <parameters>$(find ${config_file_package})/${config_file_path}</parameters>
+        </plugin>
+      </xacro:unless>
+    </gazebo>
+  </xacro:macro>
   <xacro:macro name="diffdrive_gazebo" params="publish_tf publish_jointstate robot_namespace">
     <gazebo>

Commit message: controller managerが起動するように変更 (#43)
Co-authored-by: Shota Aoki <s.aoki@rt-net.jp>

File: urdf/raspimouse.urdf.xacro (robot description, xacro)
@@ -11,6 +11,8 @@
   <xacro:arg name="jointstate" default="true" />
   <xacro:arg name="robot_namespace" default="/" />
-  <xacro:arg name="diffdrive_namespace" default="/" />
   <xacro:arg name="sensor_namespace" default="raspimouse_on_gazebo" />
+  <xacro:arg name="use_gazebo" default="false" />
+  <xacro:arg name="gz_control_config_package" default="" />
+  <xacro:arg name="gz_control_config_file_path" default="" />
   <material name="black">
     <color rgba="0.2 0.2 0.2 1.0"/>
@@ -21,4 +23,5 @@
   <xacro:include filename="$(find raspimouse_description)/urdf/wheel/wheel.urdf.xacro" />
   <xacro:include filename="$(find raspimouse_description)/urdf/wheel/diffdrive.gazebo.xacro" />
+  <xacro:include filename="$(find raspimouse_description)/urdf/wheel/diffdrive.gazebo_ros2_control.xacro" />
   <xacro:include filename="$(find raspimouse_description)/urdf/sensors/lightsens.urdf.xacro" />
   <xacro:include filename="$(find raspimouse_description)/urdf/sensors/lidar.urdf.xacro" />
@@ -81,4 +84,14 @@
   </xacro:if>
   <!-- =============== Gazebo =============== -->
+  <xacro:if value="$(arg use_gazebo)">
+    <xacro:gazebo_diffdrive_settings
+      use_gazebo="$(arg use_gazebo)"
+      config_file_package="$(arg gz_control_config_package)"
+      config_file_path="$(arg gz_control_config_file_path)" />
+    <xacro:diffdrive_gazebo_ros2_control_settings
+      name_hardware="GazeboSystem"
+      name_right_wheel_joint="right_wheel_joint"
+      name_left_wheel_joint="left_wheel_joint" />
+  </xacro:if>
   <xacro:if value="$(arg gazebo_plugin)">
     <gazebo>
@@ -113,7 +126,4 @@
       <xacro:lidar_gazebo sensor_link_name="$(arg lidar_frame)" base_rad="0" rad_range="6.28" min_range="0.15" max_range="12" />
     </xacro:if>
-    <!-- DiffDriveController -->
-    <xacro:diffdrive_gazebo publish_tf="$(arg tf)" publish_jointstate="$(arg jointstate)"
-      robot_namespace="$(arg diffdrive_namespace)" />
   </xacro:if>
   <raspimouse_on_gazebo/>

File: urdf/wheel/diffdrive.gazebo.xacro (robot description, xacro)
@@ -2,43 +2,15 @@
 <robot name="diffdrive_gazebo" xmlns:xacro="http://ros.org/wiki/xacro">
   <xacro:include filename="$(find raspimouse_description)/urdf/common.xacro" />
-  <xacro:macro name="diffdrive_gazebo" params="publish_tf publish_jointstate robot_namespace">
+  <xacro:macro name="gazebo_diffdrive_settings"
+    params="use_gazebo
+            config_file_package
+            config_file_path
+            ">
     <gazebo>
-      <plugin name="differential_drive_controller" filename="libgazebo_ros_diff_drive.so">
-        <!-- Name of robot namespace of DiffDriveController -->
-        <robotNamespace>${robot_namespace}</robotNamespace>
-        <alwaysOn>true</alwaysOn>
-        <updateRate>50</updateRate>
-        <!-- Set to true to swap right and left wheels, defaults to true -->
-        <legacyMode>false</legacyMode>
-        <rosDebugLevel>na</rosDebugLevel>
-        <!-- Name of left joint, defaults to `left_joint` -->
-        <leftJoint>left_wheel_joint</leftJoint>
-        <!-- Name of right joint, defaults to `right_joint` -->
-        <rightJoint>right_wheel_joint</rightJoint>
-        <robotBaseFrame>base_footprint</robotBaseFrame>
-        <!-- Topic to receive geometry_msgs/Twist message commands, defaults to `cmd_vel` -->
-        <commandTopic>cmd_vel</commandTopic>
-        <!-- Topic to publish nav_msgs/Odometry messages, defaults to `odom` -->
-        <odometryTopic>odom</odometryTopic>
-        <!-- Odometry frame, defaults to `odom` -->
-        <odometryFrame>odom</odometryFrame>
-        <!-- Odometry source, 0 for ENCODER, 1 for WORLD, defaults to WORLD -->
-        <odometrySource>world</odometrySource>
-        <!-- Phisical wheel params -->
-        <wheelSeparation>${wheel_separation}</wheelSeparation>
-        <wheelDiameter>${wheel_radius*2.0}</wheelDiameter>
-        <!-- Maximum torque which the wheels can produce, in Nm, defaults to 5 Nm -->
-        <wheelTorque>500</wheelTorque>
-        <!-- Wheel acceleration, in rad/s^2, defaults to 0.0 rad/s^2 -->
-        <wheelAcceleration>0</wheelAcceleration>
-        <!-- Set to true to publish /odom (nav_msgs::Odometry), defaults to true -->
-        <publishTf>${publish_tf}</publishTf>
-        <!-- Set to true to publish transforms for the wheel links, defaults to false -->
-        <publishWheelTF>${publish_tf}</publishWheelTF>
-        <!-- Set to true to publish transforms for the odometry, defaults to true -->
-        <publishOdomTF>${publish_tf}</publishOdomTF>
-        <!-- Set to true to publish sensor_msgs/JointState on /joint_states for the wheel joints, defaults to false -->
-        <publishWheelJointState>${publish_jointstate}</publishWheelJointState>
-      </plugin>
+      <xacro:if value="${use_gazebo}">
+        <plugin filename="libign_ros2_control-system.so" name="ign_ros2_control::IgnitionROS2ControlPlugin">
+          <parameters>$(find ${config_file_package})/${config_file_path}</parameters>
+        </plugin>
+      </xacro:if>
     </gazebo>
   </xacro:macro>

Commit message: RGBカメラのモデルを表示できるように変更

File: urdf/raspimouse.urdf.xacro (robot description, xacro)
@@ -13,4 +13,5 @@
   <xacro:arg name="sensor_namespace" default="raspimouse_on_gazebo" />
   <xacro:arg name="use_gazebo" default="false" />
+  <xacro:arg name="use_rgb_camera" default="false" />
   <xacro:arg name="gz_control_config_package" default="" />
   <xacro:arg name="gz_control_config_file_path" default="" />
@@ -83,4 +84,15 @@
     </xacro:lidar_rp_sensor>
   </xacro:if>
+  <!-- RGB Camera -->
+  <xacro:if value="$(arg use_rgb_camera)">
+    <xacro:include filename="$(find realsense2_description)/urdf/_d435.urdf.xacro" />
+    <xacro:sensor_d435
+        parent="base_link"
+        use_nominal_extrinsics="false"
+        add_plug="false"
+        use_mesh="true">
+      <origin xyz="0.08 0.0 0.05" rpy="0 0 0"/>
+    </xacro:sensor_d435>
+  </xacro:if>
   <!-- =============== Gazebo =============== -->
   <xacro:if value="$(arg use_gazebo)">

Commit message: RGBカメラの位置を修正
Co-authored-by: Shota Aoki <s.aoki@rt-net.jp>

File: urdf/raspimouse.urdf.xacro (robot description, xacro)
@@ -92,5 +92,5 @@
         add_plug="false"
         use_mesh="true">
-      <origin xyz="0.08 0.0 0.05" rpy="0 0 0"/>
+      <origin xyz="0.08 0.0 0.055" rpy="0 0 0"/>
     </xacro:sensor_d435>
   </xacro:if>

Commit message: RGBカメラのモデルを表示できるように変更 (#45)
Co-authored-by: Shota Aoki <s.aoki@rt-net.jp>

File: urdf/raspimouse.urdf.xacro (robot description, xacro)
@@ -13,4 +13,5 @@
   <xacro:arg name="sensor_namespace" default="raspimouse_on_gazebo" />
   <xacro:arg name="use_gazebo" default="false" />
+  <xacro:arg name="use_rgb_camera" default="false" />
   <xacro:arg name="gz_control_config_package" default="" />
   <xacro:arg name="gz_control_config_file_path" default="" />
@@ -83,4 +84,15 @@
     </xacro:lidar_rp_sensor>
   </xacro:if>
+  <!-- RGB Camera -->
+  <xacro:if value="$(arg use_rgb_camera)">
+    <xacro:include filename="$(find realsense2_description)/urdf/_d435.urdf.xacro" />
+    <xacro:sensor_d435
+        parent="base_link"
+        use_nominal_extrinsics="false"
+        add_plug="false"
+        use_mesh="true">
+      <origin xyz="0.08 0.0 0.055" rpy="0 0 0"/>
+    </xacro:sensor_d435>
+  </xacro:if>
   <!-- =============== Gazebo =============== -->
   <xacro:if value="$(arg use_gazebo)">

Commit message: RGBカメラのxacroファイルを作成

File: urdf/raspimouse.urdf.xacro (robot description, xacro)
@@ -27,4 +27,5 @@
   <xacro:include filename="$(find raspimouse_description)/urdf/sensors/lightsens.urdf.xacro" />
   <xacro:include filename="$(find raspimouse_description)/urdf/sensors/lidar.urdf.xacro" />
+  <xacro:include filename="$(find raspimouse_description)/urdf/sensors/rgb_camera.xacro" />
   <!-- =============== Link & Joint =============== -->
   <!-- Base -->
@@ -84,20 +85,11 @@
     </xacro:lidar_rp_sensor>
   </xacro:if>
-  <!-- RGB Camera -->
-  <xacro:if value="$(arg use_rgb_camera)">
-    <xacro:include filename="$(find realsense2_description)/urdf/_d435.urdf.xacro" />
-    <xacro:sensor_d435
-        parent="base_link"
-        use_nominal_extrinsics="false"
-        add_plug="false"
-        use_mesh="true">
-      <origin xyz="0.08 0.0 0.055" rpy="0 0 0"/>
-    </xacro:sensor_d435>
-  </xacro:if>
   <!-- =============== Gazebo =============== -->
+  <xacro:rgb_camera_settings
+    use_gazebo="$(arg use_gazebo)"
+    use_rgb_camera="$(arg use_rgb_camera)" />
   <xacro:if value="$(arg use_gazebo)">
     <xacro:gazebo_diffdrive_settings
       use_gazebo="$(arg use_gazebo)"
-      use_rgb_camera="$(arg use_rgb_camera)"
       config_file_package="$(arg gz_control_config_package)"
       config_file_path="$(arg gz_control_config_file_path)" />

File: urdf/wheel/diffdrive.gazebo.xacro (robot description, xacro)
@@ -4,5 +4,4 @@
   <xacro:macro name="gazebo_diffdrive_settings"
     params="use_gazebo
-            use_rgb_camera
             config_file_package
             config_file_path
@@ -17,30 +16,4 @@
           <parameters>$(find ${config_file_package})/${config_file_path}</parameters>
         </plugin>
-	<plugin filename="ignition-gazebo-sensors-system" name="ignition::gazebo::systems::Sensors">
-        <render_engine>ogre2</render_engine>
-      </plugin>
-      </xacro:if>
-    </gazebo>
-    <gazebo reference="camera_link">
-      <xacro:if value="${use_rgb_camera}">
-        <sensor name="camera_link" type="camera">
-          <update_rate>30.0</update_rate>
-          <always_on>true</always_on>
-          <ignition_frame_id>camera_link</ignition_frame_id>
-          <pose>0 0 0 0 0 0</pose>
-	  <topic>/camera/color/image_raw</topic>
-          <camera name="rgb_camera">
-            <horizontal_fov>1.3962634</horizontal_fov>
-            <image>
-              <width>1920</width>
-              <height>1080</height>
-              <format>R8G8B8</format>
-            </image>
-            <clip>
-              <near>0.02</near>
-              <far>300</far>
-            </clip>
-          </camera>
-        </sensor>
       </xacro:if>
     </gazebo>

Commit message: Gazebo上で画像トピックを配信できるように変更 (#46)

File: urdf/raspimouse.urdf.xacro (robot description, xacro)
@@ -27,4 +27,5 @@
   <xacro:include filename="$(find raspimouse_description)/urdf/sensors/lightsens.urdf.xacro" />
   <xacro:include filename="$(find raspimouse_description)/urdf/sensors/lidar.urdf.xacro" />
+  <xacro:include filename="$(find raspimouse_description)/urdf/sensors/rgb_camera.xacro" />
   <!-- =============== Link & Joint =============== -->
   <!-- Base -->
@@ -84,16 +85,8 @@
     </xacro:lidar_rp_sensor>
   </xacro:if>
-  <!-- RGB Camera -->
-  <xacro:if value="$(arg use_rgb_camera)">
-    <xacro:include filename="$(find realsense2_description)/urdf/_d435.urdf.xacro" />
-    <xacro:sensor_d435
-        parent="base_link"
-        use_nominal_extrinsics="false"
-        add_plug="false"
-        use_mesh="true">
-      <origin xyz="0.08 0.0 0.055" rpy="0 0 0"/>
-    </xacro:sensor_d435>
-  </xacro:if>
   <!-- =============== Gazebo =============== -->
+  <xacro:rgb_camera_settings
+    use_gazebo="$(arg use_gazebo)"
+    use_rgb_camera="$(arg use_rgb_camera)" />
   <xacro:if value="$(arg use_gazebo)">
     <xacro:gazebo_diffdrive_settings
