Commit message: camera_downwardがtrueのときRGBカメラが斜め下を向くように変更

File: urdf/raspimouse.urdf.xacro (robot description, xacro)
@@ -14,4 +14,5 @@
   <xacro:arg name="use_gazebo" default="false" />
   <xacro:arg name="use_rgb_camera" default="false" />
+  <xacro:arg name="camera_downward" default="false" />
   <xacro:arg name="gz_control_config_package" default="" />
   <xacro:arg name="gz_control_config_file_path" default="" />
@@ -88,5 +89,6 @@
   <xacro:rgb_camera_settings
     use_gazebo="$(arg use_gazebo)"
-    use_rgb_camera="$(arg use_rgb_camera)" />
+    use_rgb_camera="$(arg use_rgb_camera)"
+    camera_downward="$(arg camera_downward)" />
   <xacro:if value="$(arg use_gazebo)">
     <xacro:gazebo_diffdrive_settings

File: urdf/sensors/rgb_camera.xacro (robot description, xacro)
@@ -5,14 +5,26 @@
     params="use_gazebo
             use_rgb_camera
+            camera_downward
             ">
   <xacro:if value="$(arg use_rgb_camera)">
     <xacro:include filename="$(find realsense2_description)/urdf/_d435.urdf.xacro" />
-    <xacro:sensor_d435
+    <xacro:if value="$(arg camera_downward)">
+      <xacro:sensor_d435
         parent="base_link"
         use_nominal_extrinsics="false"
         add_plug="false"
         use_mesh="true">
-      <origin xyz="0.08 0.0 0.055" rpy="0 0 0"/>
-    </xacro:sensor_d435>
+          <origin xyz="0.08 0.0 0.055" rpy="0 0.523 0"/>
+      </xacro:sensor_d435>
+    </xacro:if>
+    <xacro:unless value="$(arg camera_downward)">
+      <xacro:sensor_d435
+        parent="base_link"
+        use_nominal_extrinsics="false"
+        add_plug="false"
+        use_mesh="true">
+          <origin xyz="0.08 0.0 0.055" rpy="0 0 0"/>
+      </xacro:sensor_d435>
+    </xacro:unless>
   </xacro:if>
   <xacro:if value="${use_gazebo}">
@@ -22,25 +34,50 @@
       </plugin>
     </gazebo>
-    <gazebo reference="camera_link">
-      <sensor name="camera_link" type="camera">
-        <update_rate>30.0</update_rate>
-        <always_on>true</always_on>
-        <ignition_frame_id>camera_link</ignition_frame_id>
-        <pose>0 0 0 0 0 0</pose>
-        <topic>/camera/color/image_raw</topic>
-        <camera name="rgb_camera">
-          <horizontal_fov>1.20428</horizontal_fov>
-          <image>
-            <width>1920</width>
-            <height>1080</height>
-            <format>R8G8B8</format>
-          </image>
-          <clip>
-            <near>0.02</near>
-            <far>300</far>
-          </clip>
-        </camera>
-      </sensor>
-    </gazebo>
+    <xacro:if value="${camera_downward}">
+      <gazebo reference="camera_link">
+        <sensor name="camera_link" type="camera">
+          <update_rate>30.0</update_rate>
+          <always_on>true</always_on>
+          <ignition_frame_id>camera_link</ignition_frame_id>
+          <pose>0 0 0 0 0.523 0</pose>
+          <topic>/camera/color/image_raw</topic>
+          <camera name="rgb_camera">
+            <horizontal_fov>1.20428</horizontal_fov>
+            <image>
+              <width>1920</width>
+              <height>1080</height>
+              <format>R8G8B8</format>
+            </image>
+            <clip>
+              <near>0.02</near>
+              <far>300</far>
+            </clip>
+          </camera>
+        </sensor>
+      </gazebo>
+    </xacro:if>
+    <xacro:unless value="${camera_downward}">
+      <gazebo reference="camera_link">
+        <sensor name="camera_link" type="camera">
+          <update_rate>30.0</update_rate>
+          <always_on>true</always_on>
+          <ignition_frame_id>camera_link</ignition_frame_id>
+          <pose>0 0 0 0 0 0</pose>
+          <topic>/camera/color/image_raw</topic>
+          <camera name="rgb_camera">
+            <horizontal_fov>1.20428</horizontal_fov>
+            <image>
+              <width>1920</width>
+              <height>1080</height>
+              <format>R8G8B8</format>
+            </image>
+            <clip>
+              <near>0.02</near>
+              <far>300</far>
+            </clip>
+          </camera>
+        </sensor>
+      </gazebo>
+    </xacro:unless>
   </xacro:if>
 </xacro:macro>

Commit message: シミュレータ環境でscanトピックをpublish (#52)

File: urdf/raspimouse.urdf.xacro (robot description, xacro)
@@ -124,4 +124,6 @@
       robot_namespace="$(arg sensor_namespace)"
       robotdescription_namespace="$(arg robot_namespace)" />
+  </xacro:if>
+  <xacro:if value="$(arg use_gazebo)">
     <xacro:if value="${'$(arg lidar)' == 'urg'}">
       <xacro:lidar_gazebo sensor_link_name="$(arg lidar_frame)" base_rad="0" rad_range="4.71" min_range="0.10" max_range="5.6" />

File: urdf/sensors/rgb_camera.xacro (robot description, xacro)
@@ -8,58 +8,58 @@
             camera_downward
             ">
-  <xacro:if value="$(arg use_rgb_camera)">
-    <xacro:include filename="$(find realsense2_description)/urdf/_d435.urdf.xacro" />
-    <xacro:if value="$(arg camera_downward)">
-      <xacro:sensor_d435
-        parent="base_link"
-        use_nominal_extrinsics="false"
-        add_plug="false"
-        use_mesh="true">
-          <origin xyz="0.08 0.0 0.055" rpy="0 ${DOWNWARD_CAMERA_ANGLE} 0"/>
-      </xacro:sensor_d435>
+    <xacro:if value="$(arg use_rgb_camera)">
+      <xacro:include filename="$(find realsense2_description)/urdf/_d435.urdf.xacro" />
+      <xacro:if value="$(arg camera_downward)">
+        <xacro:sensor_d435
+          parent="base_link"
+          use_nominal_extrinsics="false"
+          add_plug="false"
+          use_mesh="true">
+            <origin xyz="0.08 0.0 0.055" rpy="0 ${DOWNWARD_CAMERA_ANGLE} 0"/>
+        </xacro:sensor_d435>
+      </xacro:if>
+      <xacro:unless value="$(arg camera_downward)">
+        <xacro:sensor_d435
+          parent="base_link"
+          use_nominal_extrinsics="false"
+          add_plug="false"
+          use_mesh="true">
+            <origin xyz="0.08 0.0 0.055" rpy="0 0 0"/>
+        </xacro:sensor_d435>
+      </xacro:unless>
+      <xacro:if value="${use_gazebo}">
+        <gazebo>
+          <plugin filename="ignition-gazebo-sensors-system" name="ignition::gazebo::systems::Sensors">
+            <render_engine>ogre2</render_engine>
+          </plugin>
+        </gazebo>
+        <gazebo reference="camera_link">
+          <sensor name="camera_link" type="camera">
+            <update_rate>30.0</update_rate>
+            <always_on>true</always_on>
+            <ignition_frame_id>camera_link</ignition_frame_id>
+            <xacro:if value="${camera_downward}">
+              <pose>0 0 0 0 ${DOWNWARD_CAMERA_ANGLE} 0</pose>
+            </xacro:if>
+            <xacro:unless value="${camera_downward}">
+              <pose>0 0 0 0 0 0</pose>
+            </xacro:unless>
+            <topic>/camera/color/image_raw</topic>
+            <camera name="rgb_camera">
+              <horizontal_fov>1.20428</horizontal_fov>
+              <image>
+                <width>1920</width>
+                <height>1080</height>
+                <format>R8G8B8</format>
+              </image>
+              <clip>
+                <near>0.02</near>
+                <far>300</far>
+              </clip>
+            </camera>
+          </sensor>
+        </gazebo>
+      </xacro:if>
     </xacro:if>
-    <xacro:unless value="$(arg camera_downward)">
-      <xacro:sensor_d435
-        parent="base_link"
-        use_nominal_extrinsics="false"
-        add_plug="false"
-        use_mesh="true">
-          <origin xyz="0.08 0.0 0.055" rpy="0 0 0"/>
-      </xacro:sensor_d435>
-    </xacro:unless>
-  </xacro:if>
-  <xacro:if value="${use_gazebo}">
-    <gazebo>
-      <plugin filename="ignition-gazebo-sensors-system" name="ignition::gazebo::systems::Sensors">
-        <render_engine>ogre2</render_engine>
-      </plugin>
-    </gazebo>
-    <gazebo reference="camera_link">
-      <sensor name="camera_link" type="camera">
-        <update_rate>30.0</update_rate>
-        <always_on>true</always_on>
-        <ignition_frame_id>camera_link</ignition_frame_id>
-        <xacro:if value="${camera_downward}">
-          <pose>0 0 0 0 ${DOWNWARD_CAMERA_ANGLE} 0</pose>
-        </xacro:if>
-        <xacro:unless value="${camera_downward}">
-          <pose>0 0 0 0 0 0</pose>
-        </xacro:unless>
-        <topic>/camera/color/image_raw</topic>
-        <camera name="rgb_camera">
-          <horizontal_fov>1.20428</horizontal_fov>
-          <image>
-            <width>1920</width>
-            <height>1080</height>
-            <format>R8G8B8</format>
-          </image>
-          <clip>
-            <near>0.02</near>
-            <far>300</far>
-          </clip>
-        </camera>
-      </sensor>
-    </gazebo>
-  </xacro:if>
-</xacro:macro>
+  </xacro:macro>
 </robot>
