Commit message: Replace depricated xacro settings

File: urdf/wheel/wheel.urdf.xacro (robot description, xacro)
@@ -3,12 +3,12 @@
   <xacro:include filename="$(find raspimouse_description)/urdf/wheel/wheel.transmission.xacro"/>
   <xacro:include filename="$(find raspimouse_description)/urdf/wheel/wheel.gazebo.xacro"/>
-  <!-- <property name="wheel_radius" value="0.0239"/> -->
-  <property name="wheel_radius" value="0.0249"/>
-  <property name="wheel_length" value="0.01"/>
-  <property name="wheel_mass" value="0.0113"/>
+  <!-- <xacro:property name="wheel_radius" value="0.0239"/> -->
+  <xacro:property name="wheel_radius" value="0.0249"/>
+  <xacro:property name="wheel_length" value="0.01"/>
+  <xacro:property name="wheel_mass" value="0.0113"/>
   <xacro:macro name="wheel" params="prefix parent *joint_origin *joint_axis">
   <joint name="${prefix}_wheel_joint" type="continuous">
-    <insert_block name="joint_origin"/>
-    <insert_block name="joint_axis"/>
+    <xacro:insert_block name="joint_origin"/>
+    <xacro:insert_block name="joint_axis"/>
     <parent link="${parent}"/>
     <child link="${prefix}_wheel"/>
@@ -24,5 +24,5 @@
     </visual>
     <collision>
-      <!-- <insert_block name="joint_origin"/> -->
+      <!-- <xacro:insert_block name="joint_origin"/> -->
         <geometry>
           <!-- <cylinder radius="${wheel_radius}" length="${wheel_length}"/> -->

Commit message: Set whell joint damping and friction to zero for stable control

File: urdf/wheel/wheel.urdf.xacro (robot description, xacro)
@@ -10,5 +10,5 @@
     <limit effort="70" velocity="15"/>
     <safety_controller  k_velocity="10" />
-    <dynamics damping="1.0" friction="1.0" />
+    <dynamics damping="0.0" friction="0.0" />
   </joint>
   <link name="${prefix}_wheel">

Commit message: ホイールを表示するためにwheelリンクのdampingを0にした

File: urdf/wheel/wheel.urdf.xacro (robot description, xacro)
@@ -10,5 +10,5 @@
     <limit effort="70" velocity="15"/>
     <safety_controller  k_velocity="10" />
-    <dynamics damping="1.0" friction="1.0" />
+    <dynamics damping="0.0" friction="1.0" />
   </joint>
   <link name="${prefix}_wheel">

Commit message: diff drive controllerでホイールを操作できるようにfrictionを0にする

File: urdf/wheel/wheel.urdf.xacro (robot description, xacro)
@@ -10,5 +10,5 @@
     <limit effort="70" velocity="15"/>
     <safety_controller  k_velocity="10" />
-    <dynamics damping="0.0" friction="1.0" />
+    <dynamics damping="0.0" friction="0.0" />
   </joint>
   <link name="${prefix}_wheel">
