Commit message: xaxroのマクロの名前をdiffdrive関連のものだと分かるように変更
Co-authored-by: Shota Aoki <s.aoki@rt-net.jp>

File: urdf/wheel/diffdrive.gazebo_ros2_control.xacro (robot description, xacro)
@@ -1,5 +1,5 @@
 <?xml version="1.0"?>
 <robot xmlns:xacro="http://www.ros.org/wiki/xacro">
-  <xacro:macro name="raspimouse_gazebo_ros2_control_settings"
+  <xacro:macro name="diffdrive_gazebo_ros2_control_settings"
     params="name_hardware
             name_right_wheel_joint
