Commit message: Adds macro lidar_multi_sensor

File: urdf/sensors/lidar.urdf.xacro (robot description, xacro)
@@ -31,3 +31,31 @@
     </link>
   </xacro:macro>
+  <xacro:macro name="lidar_multi_sensor" params="sensor_link_name parent *joint_origin">
+    <joint name="${sensor_link_name}_joint" type="fixed">
+      <xacro:insert_block name="joint_origin"/>
+      <parent link="${parent}"/>
+      <child link="${sensor_link_name}"/>
+    </joint>
+    <link name="${sensor_link_name}">
+      <visual>
+        <geometry>
+          <mesh filename="package://raspimouse_description/meshes/stl/robotis-lds01.stl" scale="0.001 0.001 0.001"/>
+        </geometry>
+      </visual>
+      <collision>
+        <!-- <geometry> -->
+          <!-- <mesh filename="package://raspimouse_description/meshes/stl/robotis-lds01.stl"/> -->
+        <!-- </geometry> -->
+        <origin xyz="0 0 -0.01815" />
+        <geometry>
+          <cylinder radius="0.025" length="0.070"/>
+        </geometry>
+      </collision>
+      <inertial>
+        <mass value="0.160" />
+        <origin xyz="0 0 0" />
+        <xacro:cylinder_inertia m="0.16" r="0.025" h="0.07" />
+      </inertial>
+    </link>
+  </xacro:macro>
 </robot>

Commit message: Update collision size

File: urdf/sensors/lidar.urdf.xacro (robot description, xacro)
@@ -47,8 +47,8 @@
           <!-- <mesh filename="package://raspimouse_description/meshes/stl/robotis-lds01.stl"/> -->
         <!-- </geometry> -->
+        <geometry>
+          <cylinder radius="0.035" length="0.040"/>
+        </geometry>
         <origin xyz="0 0 -0.01815" />
-        <geometry>
-          <cylinder radius="0.025" length="0.070"/>
-        </geometry>
       </collision>
       <inertial>

Commit message: Adds legs for LDS

File: urdf/sensors/lidar.urdf.xacro (robot description, xacro)
@@ -44,4 +44,33 @@
         <material name="dark"/>
       </visual>
+      <!-- Legs -->
+      <visual>
+        <origin xyz="0.035 0.025 -0.0228" rpy="0 0 0" />
+        <geometry>
+          <cylinder length="0.02" radius="0.005" />
+        </geometry>
+        <material name="dark" />
+      </visual>
+      <visual>
+        <origin xyz="0.035 -0.025 -0.0228" rpy="0 0 0" />
+        <geometry>
+          <cylinder length="0.02" radius="0.005" />
+        </geometry>
+        <material name="dark" />
+      </visual>
+      <visual>
+        <origin xyz="-0.022 0.031 -0.0228" rpy="0 0 0" />
+        <geometry>
+          <cylinder length="0.02" radius="0.005" />
+        </geometry>
+        <material name="dark" />
+      </visual>
+      <visual>
+        <origin xyz="-0.022 -0.031 -0.0228" rpy="0 0 0" />
+        <geometry>
+          <cylinder length="0.01" radius="0.005" />
+        </geometry>
+        <material name="dark" />
+      </visual>
       <collision>
         <!-- <geometry> -->

Commit message: fix typo

File: urdf/sensors/lidar.urdf.xacro (robot description, xacro)
@@ -69,5 +69,5 @@
         <origin xyz="-0.022 -0.031 -0.0228" rpy="0 0 0" />
         <geometry>
-          <cylinder length="0.01" radius="0.005" />
+          <cylinder length="0.02" radius="0.005" />
         </geometry>
         <material name="dark" />

Commit message: Adds lidar parameter to macro lidar_multi_sensor

File: urdf/sensors/lidar.urdf.xacro (robot description, xacro)
@@ -31,5 +31,5 @@
     </link>
   </xacro:macro>
-  <xacro:macro name="lidar_multi_sensor" params="sensor_link_name parent *joint_origin">
+  <xacro:macro name="lidar_multi_sensor" params="sensor_link_name parent lidar *joint_origin">
     <joint name="${sensor_link_name}_joint" type="fixed">
       <xacro:insert_block name="joint_origin"/>

Commit message: Adds if statement. rplidar is to be added

File: urdf/sensors/lidar.urdf.xacro (robot description, xacro)
@@ -38,53 +38,55 @@
     </joint>
     <link name="${sensor_link_name}">
-      <visual>
-        <geometry>
-          <mesh filename="package://raspimouse_description/meshes/stl/robotis-lds01.stl" scale="0.001 0.001 0.001"/>
-        </geometry>
-        <material name="dark"/>
-      </visual>
-      <!-- Legs -->
-      <visual>
-        <origin xyz="0.035 0.025 -0.0228" rpy="0 0 0" />
-        <geometry>
-          <cylinder length="0.02" radius="0.005" />
-        </geometry>
-        <material name="dark" />
-      </visual>
-      <visual>
-        <origin xyz="0.035 -0.025 -0.0228" rpy="0 0 0" />
-        <geometry>
-          <cylinder length="0.02" radius="0.005" />
-        </geometry>
-        <material name="dark" />
-      </visual>
-      <visual>
-        <origin xyz="-0.022 0.031 -0.0228" rpy="0 0 0" />
-        <geometry>
-          <cylinder length="0.02" radius="0.005" />
-        </geometry>
-        <material name="dark" />
-      </visual>
-      <visual>
-        <origin xyz="-0.022 -0.031 -0.0228" rpy="0 0 0" />
-        <geometry>
-          <cylinder length="0.02" radius="0.005" />
-        </geometry>
-        <material name="dark" />
-      </visual>
-      <collision>
-        <!-- <geometry> -->
-          <!-- <mesh filename="package://raspimouse_description/meshes/stl/robotis-lds01.stl"/> -->
-        <!-- </geometry> -->
-        <geometry>
-          <cylinder radius="0.035" length="0.040"/>
-        </geometry>
-        <origin xyz="0 0 -0.01815" />
-      </collision>
-      <inertial>
-        <mass value="0.160" />
-        <origin xyz="0 0 0" />
-        <xacro:cylinder_inertia m="0.16" r="0.025" h="0.07" />
-      </inertial>
+      <xacro:if value="${'$(arg lidar)' == 'lds'}">
+        <visual>
+          <geometry>
+            <mesh filename="package://raspimouse_description/meshes/stl/robotis-lds01.stl" scale="0.001 0.001 0.001"/>
+          </geometry>
+          <material name="dark"/>
+        </visual>
+        <!-- Legs -->
+        <visual>
+          <origin xyz="0.035 0.025 -0.0228" rpy="0 0 0" />
+          <geometry>
+            <cylinder length="0.02" radius="0.005" />
+          </geometry>
+          <material name="dark" />
+        </visual>
+        <visual>
+          <origin xyz="0.035 -0.025 -0.0228" rpy="0 0 0" />
+          <geometry>
+            <cylinder length="0.02" radius="0.005" />
+          </geometry>
+          <material name="dark" />
+        </visual>
+        <visual>
+          <origin xyz="-0.022 0.031 -0.0228" rpy="0 0 0" />
+          <geometry>
+            <cylinder length="0.02" radius="0.005" />
+          </geometry>
+          <material name="dark" />
+        </visual>
+        <visual>
+          <origin xyz="-0.022 -0.031 -0.0228" rpy="0 0 0" />
+          <geometry>
+            <cylinder length="0.02" radius="0.005" />
+          </geometry>
+          <material name="dark" />
+        </visual>
+        <collision>
+          <!-- <geometry> -->
+            <!-- <mesh filename="package://raspimouse_description/meshes/stl/robotis-lds01.stl"/> -->
+          <!-- </geometry> -->
+          <geometry>
+            <cylinder radius="0.035" length="0.040"/>
+          </geometry>
+          <origin xyz="0 0 -0.01815" />
+        </collision>
+        <inertial>
+          <mass value="0.160" />
+          <origin xyz="0 0 0" />
+          <xacro:cylinder_inertia m="0.16" r="0.025" h="0.07" />
+        </inertial>
+      </xacro:if>
     </link>
   </xacro:macro>

Commit message: Update lidar macro

File: urdf/sensors/lidar.urdf.xacro (robot description, xacro)
@@ -31,5 +31,5 @@
     </link>
   </xacro:macro>
-  <xacro:macro name="lidar_multi_sensor" params="sensor_link_name parent lidar *joint_origin">
+  <xacro:macro name="lidar_lds_sensor" params="sensor_link_name parent lidar *joint_origin">
     <joint name="${sensor_link_name}_joint" type="fixed">
       <xacro:insert_block name="joint_origin"/>
@@ -38,55 +38,53 @@
     </joint>
     <link name="${sensor_link_name}">
-      <xacro:if value="${'$(arg lidar)' == 'lds'}">
-        <visual>
-          <geometry>
-            <mesh filename="package://raspimouse_description/meshes/stl/robotis-lds01.stl" scale="0.001 0.001 0.001"/>
-          </geometry>
-          <material name="dark"/>
-        </visual>
-        <!-- Legs -->
-        <visual>
-          <origin xyz="0.035 0.025 -0.0228" rpy="0 0 0" />
-          <geometry>
-            <cylinder length="0.02" radius="0.005" />
-          </geometry>
-          <material name="dark" />
-        </visual>
-        <visual>
-          <origin xyz="0.035 -0.025 -0.0228" rpy="0 0 0" />
-          <geometry>
-            <cylinder length="0.02" radius="0.005" />
-          </geometry>
-          <material name="dark" />
-        </visual>
-        <visual>
-          <origin xyz="-0.022 0.031 -0.0228" rpy="0 0 0" />
-          <geometry>
-            <cylinder length="0.02" radius="0.005" />
-          </geometry>
-          <material name="dark" />
-        </visual>
-        <visual>
-          <origin xyz="-0.022 -0.031 -0.0228" rpy="0 0 0" />
-          <geometry>
-            <cylinder length="0.02" radius="0.005" />
-          </geometry>
-          <material name="dark" />
-        </visual>
-        <collision>
-          <!-- <geometry> -->
-            <!-- <mesh filename="package://raspimouse_description/meshes/stl/robotis-lds01.stl"/> -->
-          <!-- </geometry> -->
-          <geometry>
-            <cylinder radius="0.035" length="0.040"/>
-          </geometry>
-          <origin xyz="0 0 -0.01815" />
-        </collision>
-        <inertial>
-          <mass value="0.160" />
-          <origin xyz="0 0 0" />
-          <xacro:cylinder_inertia m="0.16" r="0.025" h="0.07" />
-        </inertial>
-      </xacro:if>
+      <visual>
+        <geometry>
+          <mesh filename="package://raspimouse_description/meshes/stl/robotis_lds01.stl" scale="0.001 0.001 0.001"/>
+        </geometry>
+        <material name="dark"/>
+      </visual>
+      <!-- Legs -->
+      <visual>
+        <origin xyz="0.035 0.025 -0.0228" rpy="0 0 0" />
+        <geometry>
+          <cylinder length="0.02" radius="0.005" />
+        </geometry>
+        <material name="dark" />
+      </visual>
+      <visual>
+        <origin xyz="0.035 -0.025 -0.0228" rpy="0 0 0" />
+        <geometry>
+          <cylinder length="0.02" radius="0.005" />
+        </geometry>
+        <material name="dark" />
+      </visual>
+      <visual>
+        <origin xyz="-0.022 0.031 -0.0228" rpy="0 0 0" />
+        <geometry>
+          <cylinder length="0.02" radius="0.005" />
+        </geometry>
+        <material name="dark" />
+      </visual>
+      <visual>
+        <origin xyz="-0.022 -0.031 -0.0228" rpy="0 0 0" />
+        <geometry>
+          <cylinder length="0.02" radius="0.005" />
+        </geometry>
+        <material name="dark" />
+      </visual>
+      <collision>
+        <!-- <geometry> -->
+          <!-- <mesh filename="package://raspimouse_description/meshes/stl/robotis_lds01.stl"/> -->
+        <!-- </geometry> -->
+        <geometry>
+          <cylinder radius="0.035" length="0.040"/>
+        </geometry>
+        <origin xyz="0 0 -0.01815" />
+      </collision>
+      <inertial>
+        <mass value="0.160" />
+        <origin xyz="0 0 0" />
+        <xacro:cylinder_inertia m="0.16" r="0.025" h="0.07" />
+      </inertial>
     </link>
   </xacro:macro>

Commit message: Adds RPLIDAR macros

File: urdf/sensors/lidar.urdf.xacro (robot description, xacro)
@@ -31,5 +31,63 @@
     </link>
   </xacro:macro>
-  <xacro:macro name="lidar_lds_sensor" params="sensor_link_name parent lidar *joint_origin">
+  <xacro:macro name="lidar_lds_sensor" params="sensor_link_name parent *joint_origin">
+    <joint name="${sensor_link_name}_joint" type="fixed">
+      <xacro:insert_block name="joint_origin"/>
+      <parent link="${parent}"/>
+      <child link="${sensor_link_name}"/>
+    </joint>
+    <link name="${sensor_link_name}">
+      <visual>
+        <geometry>
+          <mesh filename="package://raspimouse_description/meshes/stl/robotis_lds01.stl" scale="0.001 0.001 0.001"/>
+        </geometry>
+        <material name="dark"/>
+      </visual>
+      <!-- Legs -->
+      <visual>
+        <origin xyz="0.035 0.025 -0.0228" rpy="0 0 0" />
+        <geometry>
+          <cylinder length="0.02" radius="0.005" />
+        </geometry>
+        <material name="dark" />
+      </visual>
+      <visual>
+        <origin xyz="0.035 -0.025 -0.0228" rpy="0 0 0" />
+        <geometry>
+          <cylinder length="0.02" radius="0.005" />
+        </geometry>
+        <material name="dark" />
+      </visual>
+      <visual>
+        <origin xyz="-0.022 0.031 -0.0228" rpy="0 0 0" />
+        <geometry>
+          <cylinder length="0.02" radius="0.005" />
+        </geometry>
+        <material name="dark" />
+      </visual>
+      <visual>
+        <origin xyz="-0.022 -0.031 -0.0228" rpy="0 0 0" />
+        <geometry>
+          <cylinder length="0.02" radius="0.005" />
+        </geometry>
+        <material name="dark" />
+      </visual>
+      <collision>
+        <!-- <geometry> -->
+          <!-- <mesh filename="package://raspimouse_description/meshes/stl/robotis_lds01.stl"/> -->
+        <!-- </geometry> -->
+        <geometry>
+          <cylinder radius="0.035" length="0.040"/>
+        </geometry>
+        <origin xyz="0 0 -0.01815" />
+      </collision>
+      <inertial>
+        <mass value="0.160" />
+        <origin xyz="0 0 0" />
+        <xacro:cylinder_inertia m="0.16" r="0.025" h="0.07" />
+      </inertial>
+    </link>
+  </xacro:macro>
+  <xacro:macro name="lidar_rp_sensor" params="sensor_link_name parent *joint_origin">
     <joint name="${sensor_link_name}_joint" type="fixed">
       <xacro:insert_block name="joint_origin"/>

Commit message: Adds leg visual macro for the lidars

File: urdf/sensors/lidar.urdf.xacro (robot description, xacro)
@@ -3,4 +3,34 @@
   <xacro:include filename="$(find raspimouse_description)/urdf/sensors/lidar.gazebo.xacro"/>
   <xacro:arg name="laser_visual" default="false"/>
+  <xacro:macro name="lidar_legs" params="length radius z_pos">
+    <visual>
+      <origin xyz="0.035 0.025 ${z_pos}" rpy="0 0 0" />
+      <geometry>
+        <cylinder length="${length}" radius="${radius}" />
+      </geometry>
+      <material name="black" />
+    </visual>
+    <visual>
+      <origin xyz="0.035 -0.025 ${z_pos}" rpy="0 0 0" />
+      <geometry>
+        <cylinder length="${length}" radius="${radius}" />
+      </geometry>
+      <material name="black" />
+    </visual>
+    <visual>
+      <origin xyz="-0.022 0.031 ${z_pos}" rpy="0 0 0" />
+      <geometry>
+        <cylinder length="${length}" radius="${radius}" />
+      </geometry>
+      <material name="black" />
+    </visual>
+    <visual>
+      <origin xyz="-0.022 -0.031 ${z_pos}" rpy="0 0 0" />
+      <geometry>
+        <cylinder length="${length}" radius="${radius}" />
+      </geometry>
+      <material name="black" />
+    </visual>
+  </xacro:macro>
   <xacro:macro name="lidar_urg_sensor" params="sensor_link_name parent *joint_origin">
     <joint name="${sensor_link_name}_joint" type="fixed">
@@ -44,33 +74,5 @@
         <material name="black"/>
       </visual>
-      <!-- Legs -->
-      <visual>
-        <origin xyz="0.035 0.025 -0.0228" rpy="0 0 0" />
-        <geometry>
-          <cylinder length="0.019" radius="0.005" />
-        </geometry>
-        <material name="black" />
-      </visual>
-      <visual>
-        <origin xyz="0.035 -0.025 -0.0228" rpy="0 0 0" />
-        <geometry>
-          <cylinder length="0.019" radius="0.005" />
-        </geometry>
-        <material name="black" />
-      </visual>
-      <visual>
-        <origin xyz="-0.022 0.031 -0.0228" rpy="0 0 0" />
-        <geometry>
-          <cylinder length="0.019" radius="0.005" />
-        </geometry>
-        <material name="black" />
-      </visual>
-      <visual>
-        <origin xyz="-0.022 -0.031 -0.0228" rpy="0 0 0" />
-        <geometry>
-          <cylinder length="0.019" radius="0.005" />
-        </geometry>
-        <material name="black" />
-      </visual>
+      <xacro:lidar_legs length="0.019" radius="0.005" z_pos="-0.0228"/>
       <collision>
         <!-- <geometry> -->
@@ -102,33 +104,5 @@
         <material name="black"/>
       </visual>
-      <!-- Legs -->
-      <visual>
-        <origin xyz="0.035 0.025 -0.028" rpy="0 0 0" />
-        <geometry>
-          <cylinder length="0.027" radius="0.003" />
-        </geometry>
-        <material name="black" />
-      </visual>
-      <visual>
-        <origin xyz="0.035 -0.025 -0.028" rpy="0 0 0" />
-        <geometry>
-          <cylinder length="0.027" radius="0.003" />
-        </geometry>
-        <material name="black" />
-      </visual>
-      <visual>
-        <origin xyz="-0.022 0.031 -0.028" rpy="0 0 0" />
-        <geometry>
-          <cylinder length="0.027" radius="0.003" />
-        </geometry>
-        <material name="black" />
-      </visual>
-      <visual>
-        <origin xyz="-0.022 -0.031 -0.028" rpy="0 0 0" />
-        <geometry>
-          <cylinder length="0.027" radius="0.003" />
-        </geometry>
-        <material name="black" />
-      </visual>
+      <xacro:lidar_legs length="0.027" radius="0.003" z_pos="-0.028"/>
       <collision>
         <!-- <geometry> -->

Commit message: Remove comments

File: urdf/sensors/lidar.urdf.xacro (robot description, xacro)
@@ -46,7 +46,4 @@
       </visual>
       <collision>
-        <!-- <geometry> -->
-          <!-- <mesh filename="package://raspimouse_description/meshes/dae/sensor/urg_optical_axis_center_origin.dae"/> -->
-        <!-- </geometry> -->
         <origin xyz="0 0 -0.01815" />
         <geometry>
@@ -76,7 +73,4 @@
       <xacro:lidar_legs length="0.019" radius="0.005" z_pos="-0.0228"/>
       <collision>
-        <!-- <geometry> -->
-          <!-- <mesh filename="package://raspimouse_description/meshes/stl/robotis_lds01.stl"/> -->
-        <!-- </geometry> -->
         <geometry>
           <cylinder radius="0.035" length="0.040"/>
@@ -106,7 +100,4 @@
       <xacro:lidar_legs length="0.027" radius="0.003" z_pos="-0.028"/>
       <collision>
-        <!-- <geometry> -->
-          <!-- <mesh filename="package://raspimouse_description/meshes/stl/robotis_lds01.stl"/> -->
-        <!-- </geometry> -->
         <geometry>
           <cylinder radius="0.048" length="0.055"/>

Commit message: Adjust the collision size and position of the LIDARs

File: urdf/sensors/lidar.urdf.xacro (robot description, xacro)
@@ -76,5 +76,5 @@
           <cylinder radius="0.035" length="0.040"/>
         </geometry>
-        <origin xyz="0 0 -0.01815" />
+        <origin xyz="0 0 -0.008" />
       </collision>
       <inertial>
@@ -101,7 +101,7 @@
       <collision>
         <geometry>
-          <cylinder radius="0.048" length="0.055"/>
+          <cylinder radius="0.036" length="0.042"/>
         </geometry>
-        <origin xyz="0 0 -0.01815" />
+        <origin xyz="0 0 -0.008" />
       </collision>
       <inertial>
